File: PCB/NXP/rsS485_rs232_can.sch (KiCad schematic (older format))
At the start: 50 parts, among them J2 TB_1X3, J3 DB9, J4 TB_1X3, U5 MAX3072, U6 ST3232E, U7 TJA1040, U8 PESD1CAN

Commit message: Modified Profibus termination resistors (#3). Removed backup PCB file.
Parts:
- R32, R39: value 680 -> 390
- R35: value 120 -> 220
Changed lines of the file:
@@
 Sheet 4 12
 Title "CIAA RS485 - RS232 - CAN"
-Date "18 jun 2014"
+Date "7 jul 2014"
 Rev "1.0"
 Comp ""
@@
 P 3450 2250
 F 0 "R35" V 3450 2150 30  0000 C CNN
-F 1 "120" V 3400 2150 30  0000 C CNN
+F 1 "220" V 3400 2150 30  0000 C CNN
 F 2 "~" H 3450 2250 60  0000 C CNN
 F 3 "~" H 3450 2250 60  0000 C CNN
@@
 P 3450 1450
 F 0 "R32" V 3500 1350 30  0000 C CNN
-F 1 "680" V 3450 1350 30  0000 C CNN
+F 1 "390" V 3450 1350 30  0000 C CNN
 F 2 "~" H 3450 1450 60  0000 C CNN
 F 3 "~" H 3450 1450 60  0000 C CNN
@@
 P 3450 2800
 F 0 "R39" V 3450 2700 30  0000 C CNN
-F 1 "680" V 3400 2700 30  0000 C CNN
+F 1 "390" V 3400 2700 30  0000 C CNN
 F 2 "~" H 3450 2800 60  0000 C CNN
 F 3 "~" H 3450 2800 60  0000 C CNN

Commit message: RS232 shield pads to GND (#4).
Connections:
- wire segments 147 -> 149
Changed lines of the file:
@@
 P 9350 5750
 F 0 "J3" H 9350 6300 70  0000 C CNN
-F 1 "DB9" H 9350 5200 70  0000 C CNN
+F 1 "DB9" H 9100 5200 70  0000 C CNN
 F 2 "" H 9350 5750 60  0000 C CNN
 F 3 "" H 9350 5750 60  0000 C CNN
@@
 Wire Wire Line
 	1400 2450 2050 2450
+$Comp
+L GND #PWR0112
+U 1 1 53BB0454
+P 9350 6650
+F 0 "#PWR0112" H 9350 6650 30  0001 C CNN
+F 1 "GND" H 9350 6580 30  0001 C CNN
+F 2 "" H 9350 6650 60  0000 C CNN
+F 3 "" H 9350 6650 60  0000 C CNN
+	1    9350 6650
+	1    0    0    -1
+$EndComp
+Wire Wire Line
+	9300 6550 9400 6550
+Wire Wire Line
+	9350 6550 9350 6650
+Connection ~ 9350 6550
 $EndSCHEMATC

Commit message: Updated DB9 symbol including TH shield pins.
Parts:
- removed J3: DB9, symbol DB9
- added J3: DB9-TH, ~, symbol DB9-TH
Changed lines of the file:
@@
 Sheet 4 12
 Title "CIAA RS485 - RS232 - CAN"
-Date "10 jul 2014"
+Date "11 jul 2014"
 Rev "1.0"
 Comp ""
@@
 F 3 "~" H 6800 4650 60  0000 C CNN
 	1    6800 4650
-	1    0    0    -1
-$EndComp
-$Comp
-L DB9 J3
-U 1 1 52C5B35E
-P 9350 5750
-F 0 "J3" H 9350 6300 70  0000 C CNN
-F 1 "DB9" H 9100 5200 70  0000 C CNN
-F 2 "" H 9350 5750 60  0000 C CNN
-F 3 "" H 9350 5750 60  0000 C CNN
-	1    9350 5750
 	1    0    0    -1
 $EndComp
@@
 	9350 6550 9350 6650
 Connection ~ 9350 6550
+$Comp
+L DB9-TH J3
+U 1 1 53C01719
+P 9350 5750
+F 0 "J3" H 9350 6300 70  0000 C CNN
+F 1 "DB9-TH" H 9100 5200 70  0000 C CNN
+F 2 "~" H 9350 5750 60  0000 C CNN
+F 3 "~" H 9350 5750 60  0000 C CNN
+	1    9350 5750
+	1    0    0    -1
+$EndComp
 $EndSCHEMATC

Commit message: Current limiters changed to NSI50010 (10mA). U5 updated for profibus networks (SN65HVD1176DR).
Parts:
- U5: value MAX3072 -> SN65HVD1176DR
Other:
- note added: "RS485\nProfibus DP"
- note removed: "RS485"
Changed lines of the file:
@@
 Sheet 4 12
 Title "CIAA RS485 - RS232 - CAN"
-Date "11 jul 2014"
+Date "12 jul 2014"
 Rev "1.0"
 Comp ""
@@
 P 2550 2150
 F 0 "U5" H 2350 2400 30  0000 C CNN
-F 1 "MAX3072" H 2750 1900 30  0000 C CNN
+F 1 "SN65HVD1176DR" H 2750 1900 30  0000 C CNN
 F 2 "SOIC8" H 2550 2150 35  0001 C CIN
 F 3 "~" H 2550 2150 60  0000 C CNN
@@
 Text Notes 9500 7000 0    60   ~ 0
 RS232
-Text Notes 4950 3700 0    60   ~ 0
-RS485
+Text Notes 4750 3600 0    60   ~ 0
+RS485\nProfibus DP
 $Comp
 L R_MINI R47
