File: PCB/NXP/analog.sch (KiCad schematic (older format))
At the start: 61 parts, among them J16 TB_1X3, J17 TB_1X2, U11 MCP6024

Commit message: [ciaa-nxp] schematic layout fixed for newer versions of kicad
Parts:
- C34: symbol CP1 -> CP1-RESCUE-ciaa-nxp
- C35, C36, C37, C38, C39, C40, C41, C42, C43, C44, C91, C92, C93: symbol C -> C-RESCUE-ciaa-nxp
- R121, R122, R123, R124, R125, R126, R127, R128, R129, R130, R50, R51, R52, R53, R54, R55, R56, R57, R58, R59, R60, R61, R62, R63: symbol R -> R-RESCUE-ciaa-nxp
- ZA2, ZA3, ZA4, ZA5: symbol TVS -> TVS-RESCUE-ciaa-nxp
Changed lines of the file:
@@
 EESchema Schematic File Version 2
+LIBS:ciaa-nxp-rescue
 LIBS:power
 LIBS:device
@@
 LIBS:memory
 LIBS:xilinx
-LIBS:special
 LIBS:microcontrollers
 LIBS:dsp
@@
 LIBS:fqt13n06l
 LIBS:ciaa-nxp-cache
-EELAYER 27 0
+EELAYER 25 0
 EELAYER END
 $Descr A4 11693 8268
@@
 $EndDescr
 $Comp
-L C C36
+L C-RESCUE-ciaa-nxp C36
 U 1 1 52C09F11
 P 3200 1750
@@
 $EndComp
 $Comp
-L TVS ZA2
+L TVS-RESCUE-ciaa-nxp ZA2
 U 1 1 52C0BFC0
 P 3600 1800
@@
 $EndComp
 $Comp
-L R R51
+L R-RESCUE-ciaa-nxp R51
 U 1 1 52C410AD
 P 8300 1650
@@
 $EndComp
 $Comp
-L CP1 C34
+L CP1-RESCUE-ciaa-nxp C34
 U 1 1 52C4213E
 P 7750 1000
@@
 $EndComp
 $Comp
-L C C35
+L C-RESCUE-ciaa-nxp C35
 U 1 1 52C4214D
 P 7750 1250
@@
 $EndComp
 $Comp
-L GNDA #PWR0200
+L GNDA-RESCUE-ciaa-nxp #PWR0200
 U 1 1 52C42244
 P 7950 1350
@@
 $EndComp
 $Comp
-L R R54
+L R-RESCUE-ciaa-nxp R54
 U 1 1 52C423F1
 P 8300 3200
@@
 $EndComp
 $Comp
-L C C39
+L C-RESCUE-ciaa-nxp C39
 U 1 1 52C42424
 P 8550 3400
@@
 $EndComp
 $Comp
-L R R57
+L R-RESCUE-ciaa-nxp R57
 U 1 1 52C43452
 P 8300 4450
@@
 $EndComp
 $Comp
-L C C41
+L C-RESCUE-ciaa-nxp C41
 U 1 1 52C4345E
 P 8550 4650
@@
 $EndComp
 $Comp
-L R R60
+L R-RESCUE-ciaa-nxp R60
 U 1 1 52C43E59
 P 8300 6000
@@
 $EndComp
 $Comp
-L C C43
+L C-RESCUE-ciaa-nxp C43
 U 1 1 52C43E65
 P 8550 6200
@@
 	8050 6350 8050 6000
 $Comp
-L C C38
+L C-RESCUE-ciaa-nxp C38
 U 1 1 52D4C8E0
 P 4400 1350
@@
 	4300 1150 4400 1150
 $Comp
-L R R53
+L R-RESCUE-ciaa-nxp R53
 U 1 1 52D4C95C
 P 4400 1800
@@
 $EndComp
 $Comp
-L R R55
+L R-RESCUE-ciaa-nxp R55
 U 1 1 52D4C99A
 P 4900 1800
@@
 $EndComp
 $Comp
-L R R50
+L R-RESCUE-ciaa-nxp R50
 U 1 1 52D4C9C5
 P 5250 950
@@
 $EndComp
 $Comp
-L R R52
+L R-RESCUE-ciaa-nxp R52
 U 1 1 52D4C9D4
 P 5850 1250
@@
 Connection ~ 4400 1150
 $Comp
-L R R56
+L R-RESCUE-ciaa-nxp R56
 U 1 1 52D4CAA4
 P 5850 1800
@@
 Connection ~ 4400 2050
 Connection ~ 5850 1550
-Text Notes 600  600  0    60   ~ 0
+Text Notes 650  800  0    60   ~ 0
 0-10V: Jumper abierto, SPDT en 1-2.\n0-20mA: Jumper cerrado, SPDT en 2-3.
 $Comp
@@
 	7050 6350 8050 6350
 $Comp
-L C C42
+L C-RESCUE-ciaa-nxp C42
 U 1 1 52D75247
 P 3200 3300
@@
 $EndComp
 $Comp
-L TVS ZA3
+L TVS-RESCUE-ciaa-nxp ZA3
 U 1 1 52D7524D
 P 3600 3350
@@
 	6750 3600 6750 3250
 $Comp
-L C C40
+L C-RESCUE-ciaa-nxp C40
 U 1 1 52D75271
 P 4400 2900
@@
 	4300 2700 4400 2700
 $Comp
-L R R61
+L R-RESCUE-ciaa-nxp R61
 U 1 1 52D7527A
 P 4400 3350
@@
 $EndComp
 $Comp
-L R R62
+L R-RESCUE-ciaa-nxp R62
 U 1 1 52D75282
 P 4900 3350
@@
 $EndComp
 $Comp
-L R R58
+L R-RESCUE-ciaa-nxp R58
 U 1 1 52D7528A
 P 5250 2500
@@
 $EndComp
 $Comp
-L R R59
+L R-RESCUE-ciaa-nxp R59
 U 1 1 52D75292
 P 5850 2800
@@
 Connection ~ 4400 2700
 $Comp
-L R R63
+L R-RESCUE-ciaa-nxp R63
 U 1 1 52D7529B
 P 5850 3350
@@
 	5850 3050 5850 3100
 $Comp
-L C C91
+L C-RESCUE-ciaa-nxp C91
 U 1 1 52D752D5
 P 3200 4550
@@
 $EndComp
 $Comp
-L TVS ZA4
+L TVS-RESCUE-ciaa-nxp ZA4
 U 1 1 52D752DB
 P 3600 4600
@@
 	6750 4850 6750 4500
 $Comp
-L C C44
+L C-RESCUE-ciaa-nxp C44
 U 1 1 52D752FF
 P 4400 4150
@@
 	4300 3950 4400 3950
 $Comp
-L R R123
+L R-RESCUE-ciaa-nxp R123
 U 1 1 52D75308
 P 4400 4600
@@
 $EndComp
 $Comp
-L R R124
+L R-RESCUE-ciaa-nxp R124
 U 1 1 52D75310
 P 4900 4600
@@
 $EndComp
 $Comp
-L R R121
+L R-RESCUE-ciaa-nxp R121
 U 1 1 52D75318
 P 5250 3750
@@
 $EndComp
 $Comp
-L R R122
+L R-RESCUE-ciaa-nxp R122
 U 1 1 52D75320
 P 5850 4050
@@
 Connection ~ 4400 3950
 $Comp
-L R R125
+L R-RESCUE-ciaa-nxp R125
 U 1 1 52D75329
 P 5850 4600
@@
 	5850 4300 5850 4350
 $Comp
-L C C93
+L C-RESCUE-ciaa-nxp C93
 U 1 1 52D75363
 P 3200 6100
@@
 $EndComp
 $Comp
-L TVS ZA5
+L TVS-RESCUE-ciaa-nxp ZA5
 U 1 1 52D75369
 P 3600 6150
@@
 	6750 6400 6750 6050
 $Comp
-L C C92
+L C-RESCUE-ciaa-nxp C92
 U 1 1 52D7538D
 P 4400 5700
@@
 	4300 5500 4400 5500
 $Comp
-L R R128
+L R-RESCUE-ciaa-nxp R128
 U 1 1 52D75396
 P 4400 6150
@@
 $EndComp
 $Comp
-L R R129
+L R-RESCUE-ciaa-nxp R129
 U 1 1 52D7539E
 P 4900 6150
@@
 $EndComp
 $Comp
-L R R126
+L R-RESCUE-ciaa-nxp R126
 U 1 1 52D753A6
 P 5250 5300
@@
 $EndComp
 $Comp
-L R R127
+L R-RESCUE-ciaa-nxp R127
 U 1 1 52D753AE
 P 5850 5600
@@
 Connection ~ 4400 5500
 $Comp
-L R R130
+L R-RESCUE-ciaa-nxp R130
 U 1 1 52D753B7
 P 5850 6150
@@
 $EndComp
 $Comp
-L GNDA #PWR0206
+L GNDA-RESCUE-ciaa-nxp #PWR0206
 U 1 1 52DFB25F
 P 2900 2150
@@
 $EndComp
 $Comp
-L GNDA #PWR0207
+L GNDA-RESCUE-ciaa-nxp #PWR0207
 U 1 1 52DFB276
 P 7550 2300
@@
 $EndComp
 $Comp
-L GNDA #PWR0208
+L GNDA-RESCUE-ciaa-nxp #PWR0208
 U 1 1 52DFB8C4
 P 2900 3700
@@
 $EndComp
 $Comp
-L GNDA #PWR0209
+L GNDA-RESCUE-ciaa-nxp #PWR0209
 U 1 1 52DFB8CA
 P 8550 3600
@@
 $EndComp
 $Comp
-L GNDA #PWR0210
+L GNDA-RESCUE-ciaa-nxp #PWR0210
 U 1 1 52DFB8D0
 P 8550 4850
@@
 $EndComp
 $Comp
-L GNDA #PWR0211
+L GNDA-RESCUE-ciaa-nxp #PWR0211
 U 1 1 52DFB8D6
 P 2900 4950
@@
 $EndComp
 $Comp
-L GNDA #PWR0212
+L GNDA-RESCUE-ciaa-nxp #PWR0212
 U 1 1 52DFB8DC
 P 2900 6500
@@
 $EndComp
 $Comp
-L GNDA #PWR0213
+L GNDA-RESCUE-ciaa-nxp #PWR0213
 U 1 1 52DFB8E2
 P 8550 6400
@@
 $EndComp
 $Comp
-L C C37
+L C-RESCUE-ciaa-nxp C37
 U 1 1 52C422AE
 P 8550 1850
@@
 $EndComp
 $Comp
-L GNDA #PWR0214
+L GNDA-RESCUE-ciaa-nxp #PWR0214
 U 1 1 52DFB8E8
 P 8550 2050
@@
 $EndComp
 $Comp
-L GNDA #PWR0215
+L GNDA-RESCUE-ciaa-nxp #PWR0215
 U 1 1 52F6F94E
 P 1500 3550
