File: PCB/NXP/analog_out.sch (KiCad schematic (older format))
At the start: 17 parts, among them J19 TB_1X2, Q1 PBSS5240XF, Q14 BC817-40, U18 LM358

Commit message: [ciaa-nxp] schematic layout fixed for newer versions of kicad
Parts:
- C46, C88: symbol C -> C-RESCUE-ciaa-nxp
- R105, R107, R109, R80, R82, R83: symbol R -> R-RESCUE-ciaa-nxp
- U18: symbol LM358 -> LM358-RESCUE-ciaa-nxp
Changed lines of the file:
@@
 EESchema Schematic File Version 2
+LIBS:ciaa-nxp-rescue
 LIBS:power
 LIBS:device
@@
 LIBS:memory
 LIBS:xilinx
-LIBS:special
 LIBS:microcontrollers
 LIBS:dsp
@@
 LIBS:fqt13n06l
 LIBS:ciaa-nxp-cache
-EELAYER 27 0
+EELAYER 25 0
 EELAYER END
 $Descr A4 11693 8268
@@
 $EndComp
 $Comp
-L C C46
+L C-RESCUE-ciaa-nxp C46
 U 1 1 532CFB21
 P 4750 2200
@@
 $EndComp
 $Comp
-L GNDA #PWR0217
+L GNDA-RESCUE-ciaa-nxp #PWR0217
 U 1 1 532CFB46
 P 4450 3300
@@
 	4450 3250 4450 3300
 $Comp
-L GNDA #PWR0218
+L GNDA-RESCUE-ciaa-nxp #PWR0218
 U 1 1 532CFB6F
 P 5000 2200
@@
 	4950 2200 5000 2200
 $Comp
-L R R80
+L R-RESCUE-ciaa-nxp R80
 U 1 1 532D06D7
 P 4500 3600
@@
 $EndComp
 $Comp
-L R R82
+L R-RESCUE-ciaa-nxp R82
 U 1 1 532D06DF
 P 3750 3950
@@
 $EndComp
 $Comp
-L GNDA #PWR0219
+L GNDA-RESCUE-ciaa-nxp #PWR0219
 U 1 1 532D06E5
 P 3750 4250
@@
 DAC_OUT
 $Comp
-L LM358 U18
+L LM358-RESCUE-ciaa-nxp U18
 U 1 1 532A70D2
 P 4550 2850
@@
 	8300 3250 8450 3250
 $Comp
-L GNDA #PWR0220
+L GNDA-RESCUE-ciaa-nxp #PWR0220
 U 1 1 532A8008
 P 8350 3500
@@
 $EndComp
 $Comp
-L LM358 U18
+L LM358-RESCUE-ciaa-nxp U18
 U 2 1 532BC753
 P 6200 2700
@@
 	5050 2850 5100 2850
 $Comp
-L R R107
+L R-RESCUE-ciaa-nxp R107
 U 1 1 532C8188
 P 5400 3300
@@
 Connection ~ 5400 3600
 $Comp
-L R R105
+L R-RESCUE-ciaa-nxp R105
 U 1 1 532C81C4
 P 5400 2250
@@
 	7100 2350 7100 2500
 $Comp
-L R R83
+L R-RESCUE-ciaa-nxp R83
 U 1 1 532C827F
 P 7100 2100
@@
 	5400 3550 5400 3600
 $Comp
-L R R109
+L R-RESCUE-ciaa-nxp R109
 U 1 1 532CE4DA
 P 7550 2100
@@
 $EndComp
 $Comp
-L GNDA #PWR0222
+L GNDA-RESCUE-ciaa-nxp #PWR0222
 U 1 1 532CECA5
 P 7550 2350
@@
 Connection ~ 7350 3250
 $Comp
-L GNDA #PWR0223
+L GNDA-RESCUE-ciaa-nxp #PWR0223
 U 1 1 532CF8E2
 P 7450 3400
@@
 	7450 3050 7450 3100
 $Comp
-L C C88
+L C-RESCUE-ciaa-nxp C88
 U 1 1 532CF934
 P 6650 3200
@@
 $EndComp
 $Comp
-L GNDA #PWR0224
+L GNDA-RESCUE-ciaa-nxp #PWR0224
 U 1 1 532CF93A
 P 6650 3400
