File: PCB/NXP/usb_otg.sch (KiCad schematic (older format))
At the start: 11 parts, among them J6 ZX62-AB-5PA, U10 MIC2025-2YM, U9 PRTR5V0U2X

Commit message: [ciaa-nxp] schematic layout fixed for newer versions of kicad
Parts:
- C32, C33: symbol C -> C-RESCUE-ciaa-nxp
- R48, R49: symbol R -> R-RESCUE-ciaa-nxp
Changed lines of the file:
@@
 EESchema Schematic File Version 2
+LIBS:ciaa-nxp-rescue
 LIBS:power
 LIBS:device
@@
 LIBS:memory
 LIBS:xilinx
-LIBS:special
 LIBS:microcontrollers
 LIBS:dsp
@@
 LIBS:fqt13n06l
 LIBS:ciaa-nxp-cache
-EELAYER 27 0
+EELAYER 25 0
 EELAYER END
 $Descr A4 11693 8268
@@
 NoConn ~ 2050 5000
 $Comp
-L GND #PWR0117
+L GND-RESCUE-ciaa-nxp #PWR0117
 U 1 1 52BC3261
 P 1750 5000
@@
 Connection ~ 3950 4600
 $Comp
-L GND #PWR0119
+L GND-RESCUE-ciaa-nxp #PWR0119
 U 1 1 52BC329E
 P 3950 5250
@@
 $EndComp
 $Comp
-L GND #PWR0120
+L GND-RESCUE-ciaa-nxp #PWR0120
 U 1 1 52BC3F9D
 P 5150 5000
@@
 $EndComp
 $Comp
-L C C32
+L C-RESCUE-ciaa-nxp C32
 U 1 1 52BC40A7
 P 7550 4650
@@
 	7550 4950 7550 4850
 $Comp
-L GND #PWR0121
+L GND-RESCUE-ciaa-nxp #PWR0121
 U 1 1 52BC411A
 P 7550 4950
@@
 $EndComp
 $Comp
-L GND #PWR0122
+L GND-RESCUE-ciaa-nxp #PWR0122
 U 1 1 52BC4129
 P 7200 4950
@@
 	1    0    0    -1
 $EndComp
-Connection ~ 8800 3300
 Wire Wire Line
 	10150 3400 9400 3400
 Wire Wire Line
 	9400 3400 9400 3450
-Connection ~ 9000 3450
 Wire Wire Line
 	10150 3500 9500 3500
 Wire Wire Line
 	9500 3500 9500 3600
-Connection ~ 8900 3600
 Wire Wire Line
 	10150 3600 9600 3600
@@
 	9700 3700 9700 4950
 $Comp
-L GND #PWR0123
+L GND-RESCUE-ciaa-nxp #PWR0123
 U 1 1 52BC45E9
 P 9700 4950
@@
 Connection ~ 10050 3900
 $Comp
-L C C33
+L C-RESCUE-ciaa-nxp C33
 U 1 1 52BC4969
 P 3950 4900
@@
 $EndComp
 $Comp
-L R R49
+L R-RESCUE-ciaa-nxp R49
 U 1 1 52C9D8D3
 P 1450 4600
@@
 Connection ~ 1750 4600
 $Comp
-L +3.3V #PWR0124
+L +3.3V-RESCUE-ciaa-nxp #PWR0124
 U 1 1 52C9D999
 P 1150 4600
@@
 	1150 4600 1200 4600
 $Comp
-L R R48
+L R-RESCUE-ciaa-nxp R48
 U 1 1 52C9D9F8
 P 1450 4400
@@
 $EndComp
 $Comp
-L GND #PWR0125
+L GND-RESCUE-ciaa-nxp #PWR0125
 U 1 1 52C9DA03
 P 1150 4450
