File: PCB/EDU-NXP/rsS485_can.sch (KiCad schematic (older format))
At the start: 22 parts, among them J1 TB_1X3, U1 SN65HVD1176DR

Commit message: Logo Open Hardware
Changed lines of the file:
@@
 Sheet 2 7
 Title "EDU CIAA RS485"
-Date "22 oct 2014"
+Date "26 oct 2014"
 Rev "1.0"
 Comp ""
@@
 $EndComp
 $Comp
-L GND #PWR4
+L GND #PWR01
 U 1 1 52C5B34B
 P 4650 3550
-F 0 "#PWR4" H 4650 3550 30  0001 C CNN
+F 0 "#PWR01" H 4650 3550 30  0001 C CNN
 F 1 "GND" H 4650 3480 30  0001 C CNN
 F 2 "" H 4650 3550 60  0000 C CNN
@@
 $EndComp
 $Comp
-L GND #PWR3
+L GND #PWR02
 U 1 1 52C5B37F
 P 4600 4450
-F 0 "#PWR3" H 4600 4450 30  0001 C CNN
+F 0 "#PWR02" H 4600 4450 30  0001 C CNN
 F 1 "GND" H 4600 4380 30  0001 C CNN
 F 2 "" H 4600 4450 60  0000 C CNN
@@
 $EndComp
 $Comp
-L GND #PWR2
+L GND #PWR03
 U 1 1 52C5B381
 P 4300 4450
-F 0 "#PWR2" H 4300 4450 30  0001 C CNN
+F 0 "#PWR03" H 4300 4450 30  0001 C CNN
 F 1 "GND" H 4300 4380 30  0001 C CNN
 F 2 "" H 4300 4450 60  0000 C CNN
@@
 $EndComp
 $Comp
-L GND #PWR6
+L GND #PWR04
 U 1 1 52C5B386
 P 5200 4650
-F 0 "#PWR6" H 5200 4650 30  0001 C CNN
+F 0 "#PWR04" H 5200 4650 30  0001 C CNN
 F 1 "GND" H 5200 4580 30  0001 C CNN
 F 2 "" H 5200 4650 60  0000 C CNN
@@
 	7450 4600 7450 4450
 $Comp
-L +5V #PWR5
+L +5V #PWR05
 U 1 1 534DAB60
 P 5200 3150
-F 0 "#PWR5" H 5200 3240 20  0001 C CNN
+F 0 "#PWR05" H 5200 3240 20  0001 C CNN
 F 1 "+5V" H 5200 3240 30  0000 C CNN
 F 2 "" H 5200 3150 60  0000 C CNN
@@
 $EndComp
 $Comp
-L +5V #PWR7
+L +5V #PWR06
 U 1 1 534DB2EC
 P 5850 2950
-F 0 "#PWR7" H 5850 3040 20  0001 C CNN
+F 0 "#PWR06" H 5850 3040 20  0001 C CNN
 F 1 "+5V" H 5850 3040 30  0000 C CNN
 F 2 "" H 5850 2950 60  0000 C CNN
@@
 $EndComp
 $Comp
-L +5V #PWR8
+L +5V #PWR07
 U 1 1 534DB96D
 P 6100 2950
-F 0 "#PWR8" H 6100 3040 20  0001 C CNN
+F 0 "#PWR07" H 6100 3040 20  0001 C CNN
 F 1 "+5V" H 6100 3040 30  0000 C CNN
 F 2 "" H 6100 2950 60  0000 C CNN
@@
 $EndComp
 $Comp
-L +3.3V #PWR1
+L +3.3V #PWR08
 U 1 1 534DC77A
 P 4150 3350
-F 0 "#PWR1" H 4150 3310 30  0001 C CNN
+F 0 "#PWR08" H 4150 3310 30  0001 C CNN
 F 1 "+3.3V" H 4150 3460 30  0000 C CNN
 F 2 "" H 4150 3350 60  0000 C CNN
@@
 Connection ~ 4150 3650
 $Comp
-L LOGO #G2
+L LOGO #G4
 U 1 1 53C3FC4E
 P 10600 6600
-F 0 "#G2" H 10600 6197 60  0001 C CNN
+F 0 "#G4" H 10600 6197 60  0001 C CNN
 F 1 "LOGO" H 10600 7003 60  0001 C CNN
 F 2 "" H 10600 6600 60  0000 C CNN
@@
 $EndComp
 $Comp
-L GND #PWR9
+L GND #PWR09
 U 1 1 540092A7
 P 6850 3050
-F 0 "#PWR9" H 6850 3050 30  0001 C CNN
+F 0 "#PWR09" H 6850 3050 30  0001 C CNN
 F 1 "GND" H 6850 2980 30  0001 C CNN
 F 2 "" H 6850 3050 60  0000 C CNN
@@
 Wire Wire Line
 	6850 2950 6850 3050
+$Comp
+L OSHWA #G3
+U 1 1 544CF17C
+P 9700 6700
+F 0 "#G3" H 9670 7100 60  0001 C CNN
+F 1 "OSHWA" H 9700 7003 60  0001 C CNN
+F 2 "~" H 9700 6700 60  0000 C CNN
+F 3 "~" H 9700 6700 60  0000 C CNN
+	1    9700 6700
+	1    0    0    -1
+$EndComp
 $EndSCHEMATC

Commit message: Se cargaron los datasheets en EDU-NXP/Datasheets y en el BOM
Parts:
- R1: footprint ~ -> SM0805; Footprint estándar (none) -> 0805; Path datasheet (none) -> ...PCB\\EDU-NXP\\Datasheets
Changed lines of the file:
@@
 Sheet 2 7
 Title "EDU CIAA RS485"
-Date "27 nov 2014"
+Date "28 nov 2014"
 Rev "1.0"
 Comp ""
@@
 F 0 "R1" V 4150 3400 30  0000 C CNN
 F 1 "4K7" V 4100 3400 30  0000 C CNN
-F 2 "~" H 4150 3500 60  0000 C CNN
+F 2 "SM0805" H 4150 3500 60  0001 C CNN
 F 3 "~" H 4150 3500 60  0000 C CNN
+F 4 "~" H 4150 3500 60  0001 C CNN "Descripción"
+F 5 "~" H 4150 3500 60  0001 C CNN "Fabricante"
+F 6 "~" H 4150 3500 60  0001 C CNN "Nro de parte"
+F 7 "...PCB\\EDU-NXP\\Datasheets" H 4150 3500 60  0001 C CNN "Path datasheet"
+F 8 "~" H 4150 3500 60  0001 C CNN "Digikey/Mouser"
+F 9 "0805" H 4150 3500 60  0001 C CNN "Footprint estándar"
 	1    4150 3500
 	0    -1   -1   0

Commit message: Se documentaron todos los componentes en el esquemático
Parts:
- C1: value 10uF / 6V3 -> 10uF; footprint ~ -> c_1206_tantalio; Descripción (none) -> CAP CER 10UF 16V 10% X7R 1206; Digikey (none) -> 399-3525-1-ND; Fabricante (none) -> Kemet; Footprint (none) -> 1206; Nro de parte (none) -> C1206C106K4RACTU; Path datasheet (none) -> ..PCB/EDU-CIAA/Datasheets
- C2: footprint ~ -> c_0805; Descripción (none) -> CAP CER 0.1UF 16V 10% X7R 0805; Digikey (none) -> 399-1167-1-ND; Fabricante (none) -> Kemet; Footprint (none) -> 0805; Nro de Parte (none) -> C0805C104K4RACTU; Path datasheet (none) -> ..PCB/EDU-NXP/Datasheets
- D1, D2, D3: footprint ~ -> DO-214AA(SMB); Descripción (none) -> TVS DIODE 10.2VWM 16.7VC SMB; Digikey (none) -> P6SMB12CAT3GOSCT-ND; Fabricante (none) -> ON Semiconductor; Footprint (none) -> DO-214AA, SMB; Nro de parte (none) -> P6SMB12CAT3G; Path datasheet (none) -> PCB/EDU-NXP/Datasheets
- J1: footprint (none) -> bornier3; Descripción (none) -> TERM BLOCK 5.08MM VERT 3POS PCB; Digikey (none) -> ED2610-ND; Fabricante (none) -> On Shore Technology Inc; Nro de parte (none) -> OSTTC032162; Path datasheet (none) -> ..PCB/EDU-NXP/Datasheets
- PS1, PS2: footprint ~ -> SM1210; Descripción (none) -> FUSE RESETTABLE .20A 30V HLD SMD; Digikey (none) -> MF-USMF020-2CT-ND; Fabricante (none) -> Bourns Inc.; Footprint (none) -> 1210; Nro de parte (none) -> MF-USMF020-2; Path datasheet (none) -> ..PCB/EDU-NXP/Datasheets
- R1: Descripción (none) -> RES 4.7K OHM 1/8W 5% 0805 SMD; Digikey (none) -> 1276-5544-1-ND; Fabricante (none) -> Samsung; Footprint  (none) -> 0805; Footprint estándar 0805 -> (none); Nro de parte (none) -> RC2012J472CS; Path datasheet ...PCB\\EDU-NXP\\Datasheets -> ..PCB/EDU-NXP/Datasheets
- R2: footprint ~ -> SM0805; Descricpión (none) -> RES 4.7K ohm 1/8W 5% 0805 SMD; Digikey (none) -> 1276-5544-1-ND; Fabricante (none) -> Samsung; Footprint (none) -> 0805; Numero de parte (none) -> RC2012J472CS; Path datasheet (none) -> ..PCB/EDU-NXP/Datasheets
- R3: footprint ~ -> SM0805; Descripción (none) -> RES 4.7K ohm 1/8 W 5% 0805 SMD; Digikey (none) -> 1276-5544-1-ND; Fabricante  (none) -> Samsung; Footprint (none) -> 0805; Nro de parte (none) -> RC2012J472CS; Path datasheet (none) -> ..PCB/EDU-NXP/Datasheets
- R4, R5: footprint ~ -> SM0805; Descripción (none) -> RES 100K OHM 1/8W 5% 0805 SMD; Digikey (none) -> P100KACT-ND; Fabricante (none) -> Panasonic Electronic Components; Footprint (none) -> 0805; Nro de parte (none) -> ERJ-6GEYJ104V; Path datasheet (none) -> ..PCB/EDU-NXP/Datasheets
- R6, R8: footprint ~ -> SM0805; Descripción (none) -> RES 390 OHM 1/10W .5% 0805 SMD; Digikey (none) -> RR12P390DCT-ND; Fabricante (none) -> Susumu; Footprint (none) -> 0805; Nro de parte (none) -> RR1220P-391-D; Path datasheet (none) -> ..PCB/EDU-NXP/Datasheets
- R7: footprint ~ -> SM0805; Descripción (none) -> RES 200 OHM 1/10W .5% 0805 SMD; Digikey (none) -> RR12P200DCT-ND; Fabricante (none) -> Susumu; Footprint (none) -> 0805; Nro de parte (none) -> RR1220P-201-D; Path datasheet (none) -> ..PCB/EDU-NXP/Datasheets
- R9: value 100 / 1/2W -> 100; footprint ~ -> SM0805; Descripción (none) -> RES 100 OHM 1/2W 1% 0805 SMD; Digikey (none) -> P16057CT-ND; Fabricante (none) -> Panasonic Electronic Components; Footprint (none) -> 0805; Nro de parte (none) -> ERJ-P06F1000V; Path datasheet (none) -> ..PCB/EDU-NXP/Datasheets
- U1: footprint SOIC8 -> -SOIC8; Descripción (none) -> IC RS485 PROFIBUS TXRX 8-SOIC; Digikey (none) -> 296-26337-1-ND; Fabricante (none) -> Texas Instruments; Footprint (none) -> 8-SOIC (0.154\", 3.90mm Width); Nro de parte (none) -> SN65HVD1176DR; Path datasheet (none) -> ../PCB/EDU-NXP/Datasheets
