File: PCB/EDU-NXP/usb.sch (KiCad schematic (older format))
At the start: 11 parts, among them J2 ZX62D-AB-5P8, U2 PRTR5V0U2X, U9 MIC2025

Commit message: Se documentaron todos los componentes en el esquemático
Parts:
- C3: footprint ~ -> c_1206_tantalio; Descripción (none) -> CAP CER 10UF 16V 10% X7R 1206; Digikey (none) -> 399-3525-1-ND; Fabricante (none) -> Kemet; Footprint (none) -> 1206; Nro de parte (none) -> C1206C106K4RACTU; Path datasheet (none) -> ..PCB/EDU-CIAA/Datasheets
- C4, C50: footprint ~ -> c_0805; Descripción (none) -> CAP CER 0.1UF 16V 10% X7R 0805; Digikey (none) -> 399-1167-1-ND; Fabricante (none) -> Kemet; Footprint (none) -> 0805; Nro de Parte (none) -> C0805C104K4RACTU; Path datasheet (none) -> ..PCB/EDU-NXP/Datasheets
- FB1: footprint ~ -> SM0805; Descripción (none) -> FERRITE CHIP POWER 220 OHM SMD; Digikey (none) -> 240-2392-1-ND; Fabricante (none) -> Laird-Signal Integrity Products; Footprint (none) -> 0805; Nro de parte (none) -> MI0805M221R-10; Path datasheet (none) -> ..PCB/EDU-NXP/Datasheets
- FB2: footprint ~ -> SM0805; Descripción (none) -> FERRITE 500MA 600 OHM 0805 SMD; Digikey (none) -> 240-2399-1-ND; Fabricante (none) -> Laird-Signal Integrity Products; Footprint (none) -> 0805; Nro de parte (none) -> HZ0805E601R-10; Path datasheet (none) -> ..PCB/EDU-NXP/Datasheets
- J2: footprint (none) -> USB_microAB_ZX62-AB-5P8; Descripción (none) -> CONN RCPT MCR USB AB SMD TH SHLL; Digikey (none) -> H11494CT-ND; Fabricante (none) -> Hirose Electric Co Ltd; Nro de parte (none) -> ZX62D-AB-5P8; Path datahseet (none) -> ..PCB/EDU-NXP/Datasheets
- R16, R17: footprint ~ -> SM0805; Descripción (none) -> RES 10K OHM 1/8W 5% 0805 SMD; Digikey (none) -> P10KACT-ND; Fabricante (none) -> Panasonic Electronic Components; Footprint (none) -> 0805; Nro de parte (none) -> ERJ-6GEYJ103V; Path datasheet (none) -> ..PCB/EDU-NXP/Datasheets
- TR1: footprint (none) -> SRF2012; Descripción (none) -> CHOKE COMMON MODE 90 OHM 0805; Digikey (none) -> 490-1064-2-ND; Fabricante (none) -> Murata Electronics North America; Footprint (none) -> 0805; Nro de parte (none) -> DLW21HN900SQ2L; Path datasheet (none) -> ../PCB/EDU-NXP/Datasheets
- U2: footprint ~ -> sot143B; Descripción (none) -> TVS DIODE 5.5VWM SOT143B; Digikey (none) -> 568-4140-1-ND; Fabricante (none) -> NXP Semiconductors; Footprint (none) -> SOT-143B; Nro de parte (none) -> PRTR5V0U2X,215; Path datasheet (none) -> ../PCB/EDU-NXP/Datasheets
- U9: footprint ~ -> -SOIC8; Descripción (none) -> IC SW DISTRIBUTION 1CHAN 8SOIC; Digikey (none) -> 576-1058-ND; Fabricante (none) -> Micrel Inc; Footprint (none) -> 8-SOIC; Nro de parte (none) -> MIC2025-2YM; Path datasheet (none) -> ../PCB/EDU-NXP/Datasheets
Changed lines of the file:
@@
 Sheet 3 7
 Title "EDU CIAA USB"
-Date "28 nov 2014"
+Date "6 dec 2014"
 Rev "1.0"
 Comp ""
@@
 F 0 "U2" H 5800 4950 70  0000 C CNN
 F 1 "PRTR5V0U2X" H 5800 4300 70  0000 C CNN
-F 2 "~" H 7350 4000 60  0000 C CNN
-F 3 "~" H 7350 4000 60  0000 C CNN
+F 2 "sot143B" H 7350 4000 60  0001 C CNN
+F 3 "PRTR5V0U2X.pdf" H 7350 4000 60  0001 C CNN
+F 4 "TVS DIODE 5.5VWM SOT143B" H 5800 4650 60  0001 C CNN "Descripción"
+F 5 "NXP Semiconductors" H 5800 4650 60  0001 C CNN "Fabricante"
+F 6 "PRTR5V0U2X,215" H 5800 4650 60  0001 C CNN "Nro de parte"
+F 7 "../PCB/EDU-NXP/Datasheets" H 5800 4650 60  0001 C CNN "Path datasheet"
+F 8 "568-4140-1-ND" H 5800 4650 60  0001 C CNN "Digikey"
+F 9 "SOT-143B" H 5800 4650 60  0001 C CNN "Footprint"
 	1    5800 4650
 	1    0    0    -1
@@
 F 0 "C3" H 7250 4750 40  0000 L CNN
 F 1 "10uF" H 7250 4550 40  0000 L CNN
-F 2 "~" H 7300 4500 30  0000 C CNN
-F 3 "~" H 7200 4650 300 0000 C CNN
+F 2 "c_1206_tantalio" H 4650 3350 60  0001 C CNN
+F 3 "KEM_C1002_X7R_SMD.pdf" H 4650 3350 60  0001 C CNN
+F 4 "CAP CER 10UF 16V 10% X7R 1206" H 4650 3350 60  0001 C CNN "Descripción"
+F 5 "Kemet" H 4650 3350 60  0001 C CNN "Fabricante"
+F 6 "C1206C106K4RACTU" H 4650 3350 60  0001 C CNN "Nro de parte"
+F 7 "..PCB/EDU-CIAA/Datasheets" H 4650 3350 60  0001 C CNN "Path datasheet"
+F 8 "399-3525-1-ND" H 4650 3350 60  0001 C CNN "Digikey"
+F 9 "1206" H 4650 3350 60  0001 C CNN "Footprint"
 	1    7200 4650
 	1    0    0    -1
@@
 F 0 "C4" H 7550 4750 40  0000 L CNN
 F 1 "100nF" H 7556 4565 40  0000 L CNN
-F 2 "~" H 7588 4500 30  0000 C CNN
-F 3 "~" H 7550 4650 60  0000 C CNN
+F 2 "c_0805" H 1238 5700 30  0001 C CNN
+F 3 "KEM_C1002_X7R_SMD.pdf" H 1200 5850 60  0001 C CNN
+F 4 "CAP CER 0.1UF 16V 10% X7R 0805" H 1200 5850 60  0001 C CNN "Descripción"
+F 5 "Kemet" H 1200 5850 60  0001 C CNN "Fabricante"
+F 6 "C0805C104K4RACTU" H 1200 5850 60  0001 C CNN "Nro de Parte"
+F 7 "..PCB/EDU-NXP/Datasheets" H 1200 5850 60  0001 C CNN "Path datasheet"
+F 8 "399-1167-1-ND" H 1200 5850 60  0001 C CNN "Digikey"
+F 9 "0805" H 1200 5850 60  0001 C CNN "Footprint"
 	1    7550 4650
 	1    0    0    -1
@@
 F 0 "J2" V 10450 3700 60  0000 C CNN
 F 1 "ZX62D-AB-5P8" V 10550 3700 60  0000 C CNN
-F 2 "" H 10500 3700 60  0000 C CNN
-F 3 "" H 10500 3700 60  0000 C CNN
+F 2 "USB_microAB_ZX62-AB-5P8" H 10500 3700 60  0001 C CNN
+F 3 "ZX62D-AB-5P8 RoHS.pdf" H 10500 3700 60  0001 C CNN
+F 4 "CONN RCPT MCR USB AB SMD TH SHLL" V 10500 3700 60  0001 C CNN "Descripción"
+F 5 "Hirose Electric Co Ltd" V 10500 3700 60  0001 C CNN "Fabricante"
+F 6 "ZX62D-AB-5P8" V 10500 3700 60  0001 C CNN "Nro de parte"
+F 7 "..PCB/EDU-NXP/Datasheets" V 10500 3700 60  0001 C CNN "Path datahseet"
+F 8 "H11494CT-ND" V 10500 3700 60  0001 C CNN "Digikey"
+F 9 "~" V 10500 3700 60  0001 C CNN "Footprint"
 	1    10500 3700
 	1    0    0    -1
@@
 F 0 "FB2" H 10050 4650 60  0000 C CNN
 F 1 "MMZ1608B601C" H 10050 4400 60  0000 C CNN
-F 2 "~" H 10050 4500 60  0000 C CNN
-F 3 "~" H 10050 4500 60  0000 C CNN
+F 2 "SM0805" H 8200 3300 60  0001 C CNN
+F 3 "HZ0805E601R-10.pdf" H 8200 3300 60  0001 C CNN
+F 4 "FERRITE 500MA 600 OHM 0805 SMD" H 8200 3300 60  0001 C CNN "Descripción"
+F 5 "Laird-Signal Integrity Products" H 8200 3300 60  0001 C CNN "Fabricante"
+F 6 "HZ0805E601R-10" H 8200 3300 60  0001 C CNN "Nro de parte"
+F 7 "..PCB/EDU-NXP/Datasheets" H 8200 3300 60  0001 C CNN "Path datasheet"
+F 8 "240-2399-1-ND" H 8200 3300 60  0001 C CNN "Digikey"
+F 9 "0805" H 8200 3300 60  0001 C CNN "Footprint"
 	1    10050 4500
 	0    -1   -1   0
@@
 F 0 "FB1" H 8200 3200 60  0000 C CNN
 F 1 "MI0805M221R-10" H 8200 3100 60  0000 C CNN
-F 2 "~" H 8200 3300 60  0000 C CNN
-F 3 "~" H 8200 3300 60  0000 C CNN
+F 2 "SM0805" H 8200 3300 60  0001 C CNN
+F 3 "MI0805M221R-10-B.pdf" H 8200 3300 60  0001 C CNN
+F 4 "FERRITE CHIP POWER 220 OHM SMD" H 8200 3300 60  0001 C CNN "Descripción"
+F 5 "Laird-Signal Integrity Products" H 8200 3300 60  0001 C CNN "Fabricante"
+F 6 "MI0805M221R-10" H 8200 3300 60  0001 C CNN "Nro de parte"
+F 7 "..PCB/EDU-NXP/Datasheets" H 8200 3300 60  0001 C CNN "Path datasheet"
+F 8 "240-2392-1-ND" H 8200 3300 60  0001 C CNN "Digikey"
+F 9 "0805" H 8200 3300 60  0001 C CNN "Footprint"
 	1    8200 3300
 	-1   0    0    1
@@
 F 0 "TR1" V 8450 4100 60  0000 C CNN
 F 1 "DLW21HN900SQ2" V 7900 4100 60  0000 C CNN
-F 2 "" H 8200 4100 60  0000 C CNN
-F 3 "" H 8200 4100 60  0000 C CNN
+F 2 "SRF2012" H 8200 4100 60  0001 C CNN
+F 3 "L0114S0133DLW21H.pdf" H 8200 4100 60  0001 C CNN
+F 4 "CHOKE COMMON MODE 90 OHM 0805" V 8200 4100 60  0001 C CNN "Descripción"
+F 5 "Murata Electronics North America" V 8200 4100 60  0001 C CNN "Fabricante"
+F 6 "DLW21HN900SQ2L" V 8200 4100 60  0001 C CNN "Nro de parte"
+F 7 "../PCB/EDU-NXP/Datasheets" V 8200 4100 60  0001 C CNN "Path datasheet"
+F 8 "490-1064-2-ND" V 8200 4100 60  0001 C CNN "Digikey"
+F 9 "0805" V 8200 4100 60  0001 C CNN "Footprint"
 	1    8200 4100
 	0    1    -1   0
@@
 F 0 "U9" H 3100 5900 60  0000 L CNN
 F 1 "MIC2025" H 2950 4650 60  0000 L CNN
-F 2 "~" H 3150 5300 60  0000 C CNN
-F 3 "~" H 3150 5300 60  0000 C CNN
+F 2 "-SOIC8" H 3150 5300 60  0001 C CNN
+F 3 "mic2025.pdf" H 3150 5300 60  0001 C CNN
+F 4 "IC SW DISTRIBUTION 1CHAN 8SOIC" H 3150 5300 60  0001 C CNN "Descripción"
+F 5 "Micrel Inc" H 3150 5300 60  0001 C CNN "Fabricante"
+F 6 "MIC2025-2YM" H 3150 5300 60  0001 C CNN "Nro de parte"
+F 7 "../PCB/EDU-NXP/Datasheets" H 3150 5300 60  0001 C CNN "Path datasheet"
+F 8 "576-1058-ND" H 3150 5300 60  0001 C CNN "Digikey"
+F 9 "8-SOIC" H 3150 5300 60  0001 C CNN "Footprint"
 	1    3150 5300
 	1    0    0    -1
@@
 F 0 "C50" H 4600 5600 40  0000 L CNN
 F 1 "100nF" H 4606 5415 40  0000 L CNN
-F 2 "~" H 4638 5350 30  0000 C CNN
-F 3 "~" H 4600 5500 60  0000 C CNN
+F 2 "c_0805" H 1238 5700 30  0001 C CNN
+F 3 "KEM_C1002_X7R_SMD.pdf" H 1200 5850 60  0001 C CNN
+F 4 "CAP CER 0.1UF 16V 10% X7R 0805" H 1200 5850 60  0001 C CNN "Descripción"
+F 5 "Kemet" H 1200 5850 60  0001 C CNN "Fabricante"
+F 6 "C0805C104K4RACTU" H 1200 5850 60  0001 C CNN "Nro de Parte"
+F 7 "..PCB/EDU-NXP/Datasheets" H 1200 5850 60  0001 C CNN "Path datasheet"
+F 8 "399-1167-1-ND" H 1200 5850 60  0001 C CNN "Digikey"
+F 9 "0805" H 1200 5850 60  0001 C CNN "Footprint"
 	1    4600 5500
 	1    0    0    -1
@@
 F 0 "R16" V 1380 4900 40  0000 C CNN
 F 1 "10k" V 1307 4901 40  0000 C CNN
-F 2 "~" V 1230 4900 30  0000 C CNN
-F 3 "~" H 1300 4900 30  0000 C CNN
+F 2 "SM0805" V 1230 4900 30  0001 C CNN
+F 3 "AOA0000CE1.pdf" H 1300 4900 30  0001 C CNN
+F 4 "RES 10K OHM 1/8W 5% 0805 SMD" V 1300 4900 60  0001 C CNN "Descripción"
+F 5 "Panasonic Electronic Components" V 1300 4900 60  0001 C CNN "Fabricante"
+F 6 "ERJ-6GEYJ103V" V 1300 4900 60  0001 C CNN "Nro de parte"
+F 7 "..PCB/EDU-NXP/Datasheets" V 1300 4900 60  0001 C CNN "Path datasheet"
+F 8 "P10KACT-ND" V 1300 4900 60  0001 C CNN "Digikey"
+F 9 "0805" V 1300 4900 60  0001 C CNN "Footprint"
 	1    1300 4900
 	-1   0    0    1
@@
 F 0 "R17" V 2080 4500 40  0000 C CNN
 F 1 "10k" V 2007 4501 40  0000 C CNN
-F 2 "~" V 1930 4500 30  0000 C CNN
-F 3 "~" H 2000 4500 30  0000 C CNN
+F 2 "SM0805" V 1230 4900 30  0001 C CNN
+F 3 "AOA0000CE1.pdf" H 1300 4900 30  0001 C CNN
+F 4 "RES 10K OHM 1/8W 5% 0805 SMD" V 1300 4900 60  0001 C CNN "Descripción"
+F 5 "Panasonic Electronic Components" V 1300 4900 60  0001 C CNN "Fabricante"
+F 6 "ERJ-6GEYJ103V" V 1300 4900 60  0001 C CNN "Nro de parte"
+F 7 "..PCB/EDU-NXP/Datasheets" V 1300 4900 60  0001 C CNN "Path datasheet"
+F 8 "P10KACT-ND" V 1300 4900 60  0001 C CNN "Digikey"
+F 9 "0805" V 1300 4900 60  0001 C CNN "Footprint"
 	1    2000 4500
 	-1   0    0    1

Commit message: ,lst actualizado
Parts:
- FB2: value MMZ1608B601C -> HZ0805E601R-10
Changed lines of the file:
@@
 Sheet 3 7
 Title "EDU CIAA USB"
-Date "6 dec 2014"
+Date "16 mar 2015"
 Rev "1.0"
 Comp ""
@@
 P 10050 4500
 F 0 "FB2" H 10050 4650 60  0000 C CNN
-F 1 "MMZ1608B601C" H 10050 4400 60  0000 C CNN
+F 1 "HZ0805E601R-10" H 10050 4400 60  0000 C CNN
 F 2 "SM0805" H 8200 3300 60  0001 C CNN
 F 3 "HZ0805E601R-10.pdf" H 8200 3300 60  0001 C CNN
