File: PCB/PIC/cpu.sch (KiCad schematic (older format))
At the start: 84 parts, among them J7 ZX62-AB-5PA, P4 CONN_6, P7 CONN_6, P9 FT_NC, SW1 SW_PUSH, U14 TXB0108, U16 PIC32MZ2048EC, U17 FT2232H, U19 93C46, U22 ASDMB-24.000MHZ-LC-T, U23 FT232RL, U24 23A1024, U25 TC25L5I32K7680, X1 12MHz

Commit message: CIAA PIC correccion FT232RL
Parts:
- removed C89, C94: 100nF, ~, symbol C
- removed P9: FT_NC, symbol CONN_13X2
- removed R143, R144: 1k, ~, symbol R
- removed R146, R147: 270, ~, symbol R
- removed U23: FT232RL, symbol FT232RL
- added GS3, GS?: GS2, GS2, symbol GS2
- added R96: 220, ~, symbol R
- C85: value 100nF -> 10nF
- R145: value 10k -> 220
Connections:
- net labels removed: FT232_RXD, FT232_TXD, USB_AUX_DM, USB_AUX_DP, VCC_33V
- wire segments 428 -> 356
- no-connect marks 39 -> 51
Other:
- moved on the sheet: C61, C62, C67, C68, C70, C71, C72, C73, C74, C75, C76, C77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

Commit message: CIAA PIC footprints done
Parts:
- removed P7: CONN_6, symbol CONN_6
- removed SW1: SW_PUSH, ~, symbol SW_PUSH
- added R188, R189, R190, R191, R192, R193, R194, R195, R196, R197, R198, R199, R200, R201, R202, R203, R204, R205, R206, R207: 10K, ~, symbol R
- added SW1: SW_PUSH_4, ~, symbol SW_PUSH_4
- added U26: MCP9700, symbol MCP9700
- gave numbers to parts that had none: 1
Connections:
- net +3.3V: now also U26.1 (VDD)
- net GND: now also U25.2 (GND), R188.2, R189.2, R190.2, R191.2, R192.2, R193.2, R194.2, R195.2, R196.2, R197.2, R198.2, R199.2, R200.2, R201.2, R202.2, R203.2, R204.2, R205.2, R206.2, R207.2, SW1.1, SW1.2, U26.3 (GND)
- net RESET: now also SW1.3, SW1.4
- net NC_100: now reaches U16.100 (ECRS/RH12)
- net NC_100: now also R207.1
- net NC_103: now reaches U16.103 (EBIA23/RH15)
- net NC_103: now also R206.1
- net NC_15: now reaches U16.15 (AN13/C1INC/RPG7/SDA4/RG7)
- net NC_15: now also R190.1
- net NC_19: now reaches U16.19 (EBIA16/RK0)
- net NC_19: now also R191.1
- net AD_TEMP: now reaches U16.2 (_EBIA5/AN34/PMA5/RA5)
- net AD_TEMP: now also U26.2 (VOUT)
- net NC_24: now reaches U16.24 (_AN26/RPE9/RE9)
- net NC_24: now also R192.1
- net NC_28: now reaches U16.28 (EBIA13/PMA13/RJ13)
- net NC_28: now also R193.1
- net NC_29: now reaches U16.29 (_EBIA11/PMA11/RJ14)
- net NC_29: now also R194.1
- net NC_30: now reaches U16.30 (EBIA0/PMA0/RJ15)
- net NC_30: now also R195.1
- net NC_4: now reaches U16.4 (_EBID6/AN16/PMD6/RE6)
- net NC_4: now also R188.1
- net NC_46: now reaches U16.46 (_RH3)
- net NC_46: now also R196.1
- net NC_47: now reaches U16.47 (_EBIA10/AN48/RPB8/PMA10/RB8)
- net NC_47: now also R197.1
- net NC_48: now reaches U16.48 (EBIA7/AN49/RPB9/PMA7/RB9)
- net NC_48: now also R198.1
- net NC_5: now reaches U16.5 (EBID7/AN15/PMD7/RE7_)
- net NC_5: now also R189.1
- net NC_50: now reaches U16.50 (AN6/RB11)
- net NC_50: now also R199.1
- net NC_51: now reaches U16.51 (_EBIA1/PMA1/RK1)
- net NC_51: now also R200.1
- net NC_52: now reaches U16.52 (_EBIA3/PMA3/RK2)
- net NC_52: now also R201.1
- net NC_62: now reaches U16.62 (AN10/RPB15/OCFB/RB15)
- net NC_62: now also R202.1
- net NC_67: now reaches U16.67 (AN42/ERXD2/RH6)
- net NC_67: now also R203.1
- net NC_68: now reaches U16.68 (EBIA4/PMA4/RH7)
- net NC_72: now reaches U16.72 (OSCO/CLKO/RC15)
- net NC_72: now also R204.1
- net NC_98: now reaches U16.98 (RPD10/SCK4/RD10)
- net NC_98: now also R205.1
- no-connect marks 51 -> 28
Other:
- note removed: "ICSP - RJ11\n"
- moved on the sheet: C47, C48, C49, C50, C51, C52, C53, C54, C55, C56, C57, C58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

Commit message: Correcciones al esquematico segun rev01
Parts:
- removed C59, C61, C62, C67, C70, C71, C72, C73, C74, C75, C76, C77, C86, C87, C90, C99: 100nF, ~, symbol C
- removed C60: 1uF, ~, symbol C
- removed C68, C78: 10uF, ~, symbol CAPAPOL
- removed C79, C81: 27p, ~, symbol C
- removed C80: 3.3uF, ~, symbol C
- removed C98: 10nF, ~, symbol C
- removed D47, D49: LED, ~, symbol LED
- removed FB11, FB7: BLM18KG221SN1, ~, symbol FILTER
- removed FB8, FB9: MMZ1608B601C, symbol FILTER
- removed GS3, GS4: GS2, GS2, symbol GS2
- removed J7: ZX62-AB-5PA, symbol CONN_9
- removed R101, R102, R103, R188, R189, R190, R191, R192, R193, R194, R195, R196, R197, R198, R199, R200, R201, R202, R203, R204, R205, R206, R207: 10K, ~, symbol R
- removed R104: 2.2K, ~, symbol R
- removed R145, R96: 220, ~, symbol R
- removed R84: 270, ~, symbol R
- removed R85: 10k, ~, symbol R
- removed R86, R87, R88, R89: 0, ~, symbol R
- removed R97: 12K, ~, symbol R
- removed R98: 1k, ~, symbol R
- removed TR1: DLW21HN900SQ2, symbol TRASF_UNIP
- removed U14: TXB0108, symbol TXB0108
- removed U17: FT2232H, symbol FT2232H
- removed U19: 93C46, symbol 93C56
- removed U24: 23A1024, symbol 23A1024
- removed X1: 12MHz, ~, symbol CRYSTAL
- C47, C48, C49, C50, C51, C52, C53, C54, C55, C56, C57, C58, C69, C82, C85: symbol C -> C-RESCUE-ciaa-pic
- P4: footprint (none) -> footprints:PIN_ARRAY_6X1
- R100, R142, R90, R93, R94, R99: symbol R -> R-RESCUE-ciaa-pic
- U16: footprint ~ -> footprints:LQFP144-M05
- U22, U25: footprint ~ -> footprints:4SMD
- U26: footprint (none) -> footprints:SOT23
Connections:
- net GNDA is gone; now on net GND: U16.42 (AVSS)
- net GPIO10 is gone; now on net RESET_ETH: U16.10 (EBIBS1/RJ10)
- net GPIO11 is gone; now on net RS232_RXD: U16.11 (_EBIA12/AN21/RPC2/PMA12/RC2)
- net GPIO16 is gone; now on net DIN2: U16.126 (EBIA21/RK7)
- net GPIO17 is gone; now on net DIN3: U16.125 (EBID10/RPF1/PMD10/RF1)
- net GPIO19 is gone; now on net RS485_TXD: U16.112 (EBID12/RPD12/PMD12/RD12)
- net GPIO20 is gone; now on net RS485_RXD: U16.111 (EBID15/RPD3/PMD15/RD3)
- net NC_4 is gone; now on net AIN1: U16.4 (_EBID6/AN16/PMD6/RE6)
- net NC_46 is gone; now on net DOUT1: U16.46 (_RH3)
- net NC_47 is gone; now on net DOUT0: U16.47 (_EBIA10/AN48/RPB8/PMA10/RB8)
- net NC_48 is gone; now on net DOUT3: U16.48 (EBIA7/AN49/RPB9/PMA7/RB9)
- net NC_5 is gone; now on net AIN3: U16.5 (EBID7/AN15/PMD7/RE7_)
- net NC_50 is gone; now on net DOUT4: U16.50 (AN6/RB11)
- net NC_51 is gone; now on net GPIO13: U16.51 (_EBIA1/PMA1/RK1)
- net NC_52 is gone; now on net GPIO2: U16.52 (_EBIA3/PMA3/RK2)
- net NC_62 is gone; now on net GPIO_AN0: U16.62 (AN10/RPB15/OCFB/RB15)
- net AD_TEMP: now also U16.144 (EBID4/AN18/PMD4/RE4); no longer U16.2 (_EBIA5/AN34/PMA5/RA5)
- net AIN0: now also U16.3 (EBID5/AN17/RPE5/PMD5/RE5_); no longer U16.36 (PGED1/AN0/RPB0/RB0)
- net AIN1: no longer U16.26 (AN4/C1INB/RB4)
- net AIN2: now also U16.1 (_AN23/RG15_); no longer U16.44 (_AN39/ETXD3/RH1)
- net AIN3: no longer U16.43 (AN38/ETXD2/RH0)
- net CAN_TD: now also U16.36 (PGED1/AN0/RPB0/RB0); no longer U16.69 (AN32/RPD14/RD14)
- net DIN0: now also U16.142 (EBID2/PMD2/RE2); no longer U16.82 (ERXD3/RH9)
- net DIN1: now also U16.143 (EBID3/RPE3/PMD3/RE3); no longer U16.83 (ECOL/RH10)
- net DIN2: no longer U16.93 (EBIA19/RK5)
- net DIN3: no longer U16.94 (EBIA20/RK6)
- net DOUT0: no longer U16.131 (_EBICS0/RJ4)
- net DOUT1: no longer U16.132 (EBICS1/RJ5)
- net DOUT2: now also U16.45 (EBIRP/RH2); no longer U16.133 (_EBICS2/RJ6)
- net DOUT3: no longer U16.134 (_EBICS3/RJ7)
- net DOUT4: no longer U16.97 (EBIA15/RPD9/PMCS2/PMA15/RD9)
- net DOUT5: now also U16.44 (_AN39/ETXD3/RH1); no longer U16.79 (SDA3/RPF2/RF2)
- net DOUT7: now also U16.43 (AN38/ETXD2/RH0); no longer U16.13 (EBIOE/AN19/RCP4/PMRD/RC4)
- net GPIO13: no longer U16.142 (EBID2/PMD2/RE2)
- net GPIO15: now also U16.93 (EBIA19/RK5); no longer U16.127 (EBID9/RPG1/PMD9/RG1)
- net GPIO2: no longer U16.45 (EBIRP/RH2)
- net GPIO7: now also U16.83 (ECOL/RH10); no longer U16.144 (EBID4/AN18/PMD4/RE4)
- net GPIO8: now also U16.82 (ERXD3/RH9); no longer U16.143 (EBID3/RPE3/PMD3/RE3)
- net GPIO_AN0: no longer U16.6 (EBIA6/AN22/RPC1/PMA6/RC1)
- net GPIO_SPI_CS: now also U16.35 (PGEC1/AN1/RPB1/RB1); no longer U16.135 (EBID0/PMD0/RE0)
- net RESET_ETH: no longer U16.138 (_EBID1/PMD1/RE1)
- net RS232_CTS: now also U16.6 (EBIA6/AN22/RPC1/PMA6/RC1); no longer U16.3 (EBID5/AN17/RPE5/PMD5/RE5_)
- net RS232_RTS: now also U16.2 (_EBIA5/AN34/PMA5/RA5); no longer U16.110 (_EBID14/RPD2/PMD14/RD2)
- net RS232_RXD: no longer U16.34 (AN2/C2INB/RPB2/RB2)
- net RS485_DIR: now also U16.110 (_EBID14/RPD2/PMD14/RD2); no longer U16.1 (_AN23/RG15_)
- net RS485_RXD: no longer U16.35 (PGEC1/AN1/RPB1/RB1)
- net RS485_TXD: no longer U16.16 (_AN12/C2IND/RPG8/SCL4/RG8)
- net SPI_SCK: now also U16.34 (AN2/C2INB/RPB2/RB2); no longer U16.109 (RPD1/SCK1/RD1)
- net GPIO09: no longer names the net of U16.12 (EBIWE/AN20/RCP3/PMWR/RC3)
- net GPIO1: no longer names the net of U16.9 (_EBIBS0/RJ12)
- net GPIO14: no longer names the net of U16.128 (EBID8/RPG0/PMD8/RG0)
- net GPIO18: no longer names the net of U16.113 (EBID13/PMD13/RD13)
- net GPIO21: no longer names the net of U16.92 (EBIA18/RK4)
- net I2S0_TX_SCK: no longer names the net of U16.86 (EBIRDY1/SDA2/RA3)
- net NC_100: no longer names the net of U16.100 (ECRS/RH12)
- net NC_103: no longer names the net of U16.103 (EBIA23/RH15)
- net NC_15: no longer names the net of U16.15 (AN13/C1INC/RPG7/SDA4/RG7)
- net NC_19: no longer names the net of U16.19 (EBIA16/RK0)
- net NC_24: no longer names the net of U16.24 (_AN26/RPE9/RE9)
- net NC_28: no longer names the net of U16.28 (EBIA13/PMA13/RJ13)
- net NC_29: no longer names the net of U16.29 (_EBIA11/PMA11/RJ14)
- net NC_30: no longer names the net of U16.30 (EBIA0/PMA0/RJ15)
- net NC_67: no longer names the net of U16.67 (AN42/ERXD2/RH6)
- net NC_68: no longer names the net of U16.68 (EBIA4/PMA4/RH7)
- net NC_72: no longer names the net of U16.72 (OSCO/CLKO/RC15)
- net NC_98: no longer names the net of U16.98 (RPD10/SCK4/RD10)
- net RPF4_SDA5: no longer names the net of U16.90 (_EBIA9/RPF4/SDA5/PMA9/RF4)
- net RPF5_SCL5: no longer names the net of U16.91 (_EBIA8/RPF5/SCL5/PMA8/RF5)
- net USB_PWR_FAULT: no longer names the net of U16.23 (AN25/RPE8/RE8)
- net Vref+: no longer names the net of U16.40 (Vref+/CVref+/AN28/RA10)
- net Vref-: no longer names the net of U16.39 (Vref-/CVref-/AN27/RA9)
- no-connect marks 28 -> 40
Other:
- note added: "CPU"
- note added: "CPU - XTAL"
- note added: "En mi KiCad veo etiquetas locales superpuestas \na pines de jerarquía. Desprolijo."
- note added: "Hoja A3 no recomendada (difícil de imprimir).\nPondría A4 portaretrato y subhoja con \nprogramador y algunas cosas.\nComo ya esta hecho así, entiendo que es difícil y trabajoso."
- note added: "ICSP"
- note added: "RESET"
- note added: "RTC - XTAL"
- note added: "S. Tempetura"
- note removed: "ICSP - IDC\n"
- moved on the sheet: C47, C48, C49, C50, C51, C52, C53, C54, C55, C56, C57, C58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

Commit message: rev02, enumeracion componentes JTAG
Other:
- note removed: "En mi KiCad veo etiquetas locales superpuestas \na pines de jerarquía. Desprolijo."
- note removed: "Hoja A3 no recomendada (difícil de imprimir).\nPondría A4 portaretrato y subhoja con \nprogramador y algunas cosas.\nComo ya esta hecho así, entiendo que es difícil y trabajoso."
Changed lines of the file:
@@
 $EndDescr
 $Comp
-L GND-RESCUE-ciaa-pic #PWR0213
+L GND-RESCUE-ciaa-pic #PWR0216
 U 1 1 52C1CF47
 P 5300 9750
-F 0 "#PWR0213" H 5300 9750 30  0001 C CNN
+F 0 "#PWR0216" H 5300 9750 30  0001 C CNN
 F 1 "GND" H 5300 9680 30  0001 C CNN
 F 2 "" H 5300 9750 60  0000 C CNN
@@
 $EndComp
 $Comp
-L GND-RESCUE-ciaa-pic #PWR0214
+L GND-RESCUE-ciaa-pic #PWR0217
 U 1 1 52C1CF54
 P 600 11000
-F 0 "#PWR0214" H 600 11000 30  0001 C CNN
+F 0 "#PWR0217" H 600 11000 30  0001 C CNN
 F 1 "GND" H 600 10930 30  0001 C CNN
 F 2 "" H 600 11000 60  0000 C CNN
@@
 $EndComp
 $Comp
-L +3.3V-RESCUE-ciaa-pic #PWR0215
+L +3.3V-RESCUE-ciaa-pic #PWR0218
 U 1 1 52C1CF55
 P 3300 10100
-F 0 "#PWR0215" H 3300 10060 30  0001 C CNN
+F 0 "#PWR0218" H 3300 10060 30  0001 C CNN
 F 1 "+3.3V" H 3300 10210 30  0000 C CNN
 F 2 "" H 3300 10100 60  0000 C CNN
@@
 $EndComp
 $Comp
-L +3.3V-RESCUE-ciaa-pic #PWR0216
+L +3.3V-RESCUE-ciaa-pic #PWR0219
 U 1 1 52C1CF61
 P 1250 2850
-F 0 "#PWR0216" H 1250 2810 30  0001 C CNN
+F 0 "#PWR0219" H 1250 2810 30  0001 C CNN
 F 1 "+3.3V" H 1250 2960 30  0000 C CNN
 F 2 "" H 1250 2850 60  0000 C CNN
@@
 $EndComp
 $Comp
-L GND-RESCUE-ciaa-pic #PWR0217
+L GND-RESCUE-ciaa-pic #PWR0220
 U 1 1 52C1CF63
 P 1250 4100
-F 0 "#PWR0217" H 1250 4100 30  0001 C CNN
+F 0 "#PWR0220" H 1250 4100 30  0001 C CNN
 F 1 "GND" H 1250 4030 30  0001 C CNN
 F 2 "" H 1250 4100 60  0000 C CNN
@@
 $EndComp
 $Comp
-L GND-RESCUE-ciaa-pic #PWR0218
+L GND-RESCUE-ciaa-pic #PWR0221
 U 1 1 52C1CF70
 P 7000 9750
-F 0 "#PWR0218" H 7000 9750 30  0001 C CNN
+F 0 "#PWR0221" H 7000 9750 30  0001 C CNN
 F 1 "GND" H 7000 9680 30  0001 C CNN
 F 2 "" H 7000 9750 60  0000 C CNN
@@
 $EndComp
 $Comp
-L +3.3V-RESCUE-ciaa-pic #PWR0223
+L +3.3V-RESCUE-ciaa-pic #PWR0222
 U 1 1 52C1CFA3
 P 3750 8850
-F 0 "#PWR0223" H 3750 8810 30  0001 C CNN
+F 0 "#PWR0222" H 3750 8810 30  0001 C CNN
 F 1 "+3.3V" H 3750 8960 30  0000 C CNN
 F 2 "" H 3750 8850 60  0000 C CNN
@@
 Text Label 1450 3250 0    60   ~ 0
 RESET
-Text Label 3700 5400 2    60   ~ 0
+Text Label 3250 5400 2    60   ~ 0
 PGEC2
 Text Label 1650 6650 0    60   ~ 0
 PGEC2
 $Comp
-L GND-RESCUE-ciaa-pic #PWR0259
+L GND-RESCUE-ciaa-pic #PWR0223
 U 1 1 5398CB6F
 P 1700 6850
-F 0 "#PWR0259" H 1700 6850 30  0001 C CNN
+F 0 "#PWR0223" H 1700 6850 30  0001 C CNN
 F 1 "GND" H 1700 6780 30  0001 C CNN
 F 2 "" H 1700 6850 60  0000 C CNN
@@
 	0    -1   -1   0
 $EndComp
-Text Label 3700 5500 2    60   ~ 0
+Text Label 3250 5500 2    60   ~ 0
 PGED2
 Text Label 1650 6750 0    60   ~ 0
 PGED2
 $Comp
-L GND-RESCUE-ciaa-pic #PWR0260
+L GND-RESCUE-ciaa-pic #PWR0224
 U 1 1 53A17893
 P 1050 9100
-F 0 "#PWR0260" H 1050 9100 30  0001 C CNN
+F 0 "#PWR0224" H 1050 9100 30  0001 C CNN
 F 1 "GND" H 1050 9030 30  0001 C CNN
 F 2 "" H 1050 9100 60  0000 C CNN
@@
 $EndComp
 $Comp
-L +3.3V-RESCUE-ciaa-pic #PWR0261
+L +3.3V-RESCUE-ciaa-pic #PWR0225
 U 1 1 53A17D5D
 P 2550 8400
-F 0 "#PWR0261" H 2550 8360 30  0001 C CNN
+F 0 "#PWR0225" H 2550 8360 30  0001 C CNN
 F 1 "+3.3V" H 2550 8510 30  0000 C CNN
 F 2 "" H 2550 8400 60  0000 C CNN
@@
 	1    0    0    -1
 $EndComp
-Text Label 3300 8500 0    60   ~ 0
+Text Label 3300 8500 2    60   ~ 0
 OSC1
 Text Label 2400 1950 0    60   ~ 0
@@
 GPIO15
 $Comp
-L +3.3V-RESCUE-ciaa-pic #PWR0266
+L +3.3V-RESCUE-ciaa-pic #PWR0226
 U 1 1 548AED7E
 P 1850 6950
-F 0 "#PWR0266" H 1850 6910 30  0001 C CNN
+F 0 "#PWR0226" H 1850 6910 30  0001 C CNN
 F 1 "+3.3V" H 1850 7060 30  0000 C CNN
 F 2 "" H 1850 6950 60  0000 C CNN
@@
 NoConn ~ 1200 1550
 $Comp
-L +3.3V-RESCUE-ciaa-pic #PWR0267
+L +3.3V-RESCUE-ciaa-pic #PWR0227
 U 1 1 548B0B5D
 P 900 1100
-F 0 "#PWR0267" H 900 1060 30  0001 C CNN
+F 0 "#PWR0227" H 900 1060 30  0001 C CNN
 F 1 "+3.3V" H 900 1210 30  0000 C CNN
 F 2 "" H 900 1100 60  0000 C CNN
@@
 $EndComp
 $Comp
-L GND-RESCUE-ciaa-pic #PWR0268
+L GND-RESCUE-ciaa-pic #PWR0228
 U 1 1 548B1668
 P 900 2150
-F 0 "#PWR0268" H 900 2150 30  0001 C CNN
+F 0 "#PWR0228" H 900 2150 30  0001 C CNN
 F 1 "GND" H 900 2080 30  0001 C CNN
 F 2 "" H 900 2150 60  0000 C CNN
@@
 $EndComp
 $Comp
-L GND-RESCUE-ciaa-pic #PWR0270
+L GND-RESCUE-ciaa-pic #PWR0229
 U 1 1 551AD1DE
 P 1350 5950
-F 0 "#PWR0270" H 1350 5950 30  0001 C CNN
+F 0 "#PWR0229" H 1350 5950 30  0001 C CNN
 F 1 "GND" H 1350 5880 30  0001 C CNN
 F 2 "" H 1350 5950 60  0000 C CNN
@@
 $EndComp
 $Comp
-L +3.3V-RESCUE-ciaa-pic #PWR0271
+L +3.3V-RESCUE-ciaa-pic #PWR0230
 U 1 1 551AD1E4
 P 1200 4850
-F 0 "#PWR0271" H 1200 4810 30  0001 C CNN
+F 0 "#PWR0230" H 1200 4810 30  0001 C CNN
 F 1 "+3.3V" H 1200 4960 30  0000 C CNN
 F 2 "" H 1200 4850 60  0000 C CNN
@@
 S. Tempetura
 $Comp
-L +3.3V-RESCUE-ciaa-pic #PWR0272
+L +3.3V-RESCUE-ciaa-pic #PWR0231
 U 1 1 575B8473
 P 4800 800
-F 0 "#PWR0272" H 4800 760 30  0001 C CNN
+F 0 "#PWR0231" H 4800 760 30  0001 C CNN
 F 1 "+3.3V" H 4800 910 30  0000 C CNN
 F 2 "" H 4800 800 60  0000 C CNN
@@
 $EndComp
 $Comp
-L +3.3VADC #PWR0273
+L +3.3VADC #PWR0232
 U 1 1 575BA482
 P 5550 800
-F 0 "#PWR0273" H 5550 920 20  0001 C CNN
+F 0 "#PWR0232" H 5550 920 20  0001 C CNN
 F 1 "+3.3VADC" H 5550 890 30  0000 C CNN
 F 2 "" H 5550 800 60  0000 C CNN
@@
 Connection ~ 1400 3450
 Wire Wire Line
-	3700 5400 3800 5400
+	3250 5400 3800 5400
 Wire Wire Line
 	1550 7050 1650 7050
@@
 	1550 6850 1700 6850
 Wire Wire Line
-	3700 5500 3800 5500
+	3250 5500 3800 5500
 Wire Wire Line
 	1550 6650 1650 6650
@@
 Text Notes 7050 850  0    138  ~ 28
 CPU
-Text Notes 300  12650 0    100  ~ 0
-Hoja A3 no recomendada (difícil de imprimir).\nPondría A4 portaretrato y subhoja con \nprogramador y algunas cosas.\nComo ya esta hecho así, entiendo que es difícil y trabajoso.
-Text Notes 200  13100 0    100  ~ 0
-En mi KiCad veo etiquetas locales superpuestas \na pines de jerarquía. Desprolijo.
 Text HLabel 7050 4100 2    60   Output ~ 0
 SQICS1
