File: PCB/PIC/fuente.sch (KiCad schematic (older format))
At the start: 19 parts, among them J18 TB_1X2, U3 LM2596-5.0, U4 NCP1117ST33T3G

Commit message: CIAA PIC footprints done
Parts:
- removed D45: PMEG3020EH, ~, symbol DIODESCH
- added D25: LED green, ~, symbol LED
- added R110: 1k, ~, symbol R
Connections:
- net +3.3V: now also R110.1
- net GND: now also D25.2 (K)
- new net: D25.1 (A), R110.2
Other:
- moved on the sheet: C16, C17, C18, D1, D2, D3, D4, D5, FB20, FB6, J18, L2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

Commit message: Correcciones al esquematico segun rev01
Parts:
- D25, D4: symbol LED -> LED-RESCUE-ciaa-pic
- R110, R22: symbol R -> R-RESCUE-ciaa-pic
- ZA1, ZA14: symbol TVS -> TVS-RESCUE-ciaa-pic
Changed lines of the file:
@@
 EESchema Schematic File Version 2
-LIBS:power
-LIBS:device
-LIBS:transistors
-LIBS:conn
-LIBS:linear
-LIBS:regul
-LIBS:74xx
-LIBS:cmos4000
-LIBS:adc-dac
-LIBS:memory
-LIBS:xilinx
-LIBS:special
-LIBS:microcontrollers
-LIBS:dsp
-LIBS:microchip
-LIBS:analog_switches
-LIBS:motorola
-LIBS:texas
-LIBS:intel
-LIBS:audio
-LIBS:interface
-LIBS:digital-audio
-LIBS:philips
-LIBS:display
-LIBS:cypress
-LIBS:siliconi
-LIBS:opto
-LIBS:atmel
-LIBS:contrib
-LIBS:valves
+LIBS:ciaa-pic-rescue
 LIBS:74LVC1G04GW
 LIBS:amesser-ad
@@
 LIBS:mcp1416
 LIBS:fqt13n06l
+LIBS:logo
+LIBS:openHW
 LIBS:ciaa-pic-cache
-EELAYER 27 0
+EELAYER 25 0
 EELAYER END
 $Descr A4 11693 8268
 encoding utf-8
-Sheet 10 12
-Title "CIAA Fuente de alimentación"
-Date "7 sep 2015"
+Sheet 10 13
+Title "CIAA-Microchip"
+Date "16 feb 2016"
 Rev "1.0"
-Comp ""
-Comment1 ""
+Comp "CIAA - COMPUTADORA INDUSTRIAL ABIERTA ARGENTINA - www.proyecto-ciaa.com.ar"
+Comment1 "Autores: Ver 'documents/CHANGES.txt'      Licencia: Ver  'documents/LICENCIA_CIAA_PIC.txt'"
 Comment2 ""
 Comment3 ""
@@
 $EndComp
 $Comp
-L GND #PWR0180
+L GND-RESCUE-ciaa-pic #PWR0189
 U 1 1 52B78A1B
 P 2900 4300
-F 0 "#PWR0180" H 2900 4300 30  0001 C CNN
+F 0 "#PWR0189" H 2900 4300 30  0001 C CNN
 F 1 "GND" H 2900 4230 30  0001 C CNN
 F 2 "" H 2900 4300 60  0000 C CNN
@@
 $EndComp
 $Comp
-L GND #PWR0181
+L GND-RESCUE-ciaa-pic #PWR0190
 U 1 1 52B78A29
 P 3750 4250
-F 0 "#PWR0181" H 3750 4250 30  0001 C CNN
+F 0 "#PWR0190" H 3750 4250 30  0001 C CNN
 F 1 "GND" H 3750 4180 30  0001 C CNN
 F 2 "" H 3750 4250 60  0000 C CNN
@@
 $EndComp
 $Comp
-L GND #PWR0182
+L GND-RESCUE-ciaa-pic #PWR0191
 U 1 1 52B78A35
 P 4600 4300
-F 0 "#PWR0182" H 4600 4300 30  0001 C CNN
+F 0 "#PWR0191" H 4600 4300 30  0001 C CNN
 F 1 "GND" H 4600 4230 30  0001 C CNN
 F 2 "" H 4600 4300 60  0000 C CNN
@@
 $EndComp
 $Comp
-L GND #PWR0183
+L GND-RESCUE-ciaa-pic #PWR0192
 U 1 1 52B78C39
 P 5850 4650
-F 0 "#PWR0183" H 5850 4650 30  0001 C CNN
+F 0 "#PWR0192" H 5850 4650 30  0001 C CNN
 F 1 "GND" H 5850 4580 30  0001 C CNN
 F 2 "" H 5850 4650 60  0000 C CNN
@@
 $EndComp
 $Comp
-L GND #PWR0184
+L GND-RESCUE-ciaa-pic #PWR0193
 U 1 1 52B78C6E
 P 6850 4650
-F 0 "#PWR0184" H 6850 4650 30  0001 C CNN
+F 0 "#PWR0193" H 6850 4650 30  0001 C CNN
 F 1 "GND" H 6850 4580 30  0001 C CNN
 F 2 "" H 6850 4650 60  0000 C CNN
@@
 $EndComp
 $Comp
-L GND #PWR0185
+L GND-RESCUE-ciaa-pic #PWR0194
 U 1 1 52B78D01
 P 7700 4750
-F 0 "#PWR0185" H 7700 4750 30  0001 C CNN
+F 0 "#PWR0194" H 7700 4750 30  0001 C CNN
 F 1 "GND" H 7700 4680 30  0001 C CNN
 F 2 "" H 7700 4750 60  0000 C CNN
@@
 $EndComp
 $Comp
-L GND #PWR0186
+L GND-RESCUE-ciaa-pic #PWR0195
 U 1 1 52B78D23
 P 8400 4650
-F 0 "#PWR0186" H 8400 4650 30  0001 C CNN
+F 0 "#PWR0195" H 8400 4650 30  0001 C CNN
 F 1 "GND" H 8400 4580 30  0001 C CNN
 F 2 "" H 8400 4650 60  0000 C CNN
@@
 $EndComp
 $Comp
-L GND #PWR0187
+L GND-RESCUE-ciaa-pic #PWR0196
 U 1 1 52C2203A
 P 4300 4350
-F 0 "#PWR0187" H 4300 4350 30  0001 C CNN
+F 0 "#PWR0196" H 4300 4350 30  0001 C CNN
 F 1 "GND" H 4300 4280 30  0001 C CNN
 F 2 "" H 4300 4350 60  0000 C CNN
@@
 $EndComp
 $Comp
-L TVS ZA1
+L TVS-RESCUE-ciaa-pic ZA1
 U 1 1 52CA0AD0
 P 4300 4100
@@
 $EndComp
 $Comp
-L LED D4
+L LED-RESCUE-ciaa-pic D4
 U 1 1 52CF8844
 P 7150 5050
@@
 $EndComp
 $Comp
-L R R22
+L R-RESCUE-ciaa-pic R22
 U 1 1 52CF884A
 P 7150 4550
@@
 $EndComp
 $Comp
-L GND #PWR0188
+L GND-RESCUE-ciaa-pic #PWR0197
 U 1 1 52CF8853
 P 7150 5400
-F 0 "#PWR0188" H 7150 5400 30  0001 C CNN
+F 0 "#PWR0197" H 7150 5400 30  0001 C CNN
 F 1 "GND" H 7150 5330 30  0001 C CNN
 F 2 "" H 7150 5400 60  0000 C CNN
@@
 	1    0    0    -1
 $EndComp
-Text Notes 4050 1250 0    60   ~ 0
+Text Notes 4050 1250 0    60   ~ 12
 Fuente de alimentación con rango aproximado de entrada de 12 a 30V (CC).\nTensiones de salida: 5V, 3A y 3.3V, 1A.\nPosibilidad de alimentar la CIAA a través del puerto USB mediante la conexión con D1.
 Wire Wire Line
@@
 	8100 4250 8700 4250
 $Comp
-L TVS ZA14
+L TVS-RESCUE-ciaa-pic ZA14
 U 1 1 52D1F0AA
 P 6550 4550
@@
 $EndComp
 $Comp
-L GND #PWR0189
+L GND-RESCUE-ciaa-pic #PWR0198
 U 1 1 52D1F0B5
 P 6550 4850
-F 0 "#PWR0189" H 6550 4850 30  0001 C CNN
+F 0 "#PWR0198" H 6550 4850 30  0001 C CNN
 F 1 "GND" H 6550 4780 30  0001 C CNN
 F 2 "" H 6550 4850 60  0000 C CNN
@@
 	9500 3850 9500 4250
 $Comp
-L +24V #PWR0190
+L +24V #PWR0199
 U 1 1 52DEA263
 P 3150 3600
-F 0 "#PWR0190" H 3150 3550 20  0001 C CNN
+F 0 "#PWR0199" H 3150 3550 20  0001 C CNN
 F 1 "+24V" H 3150 3700 30  0000 C CNN
 F 2 "" H 3150 3600 60  0000 C CNN
@@
 $EndComp
 $Comp
-L +5V #PWR0191
+L +5V #PWR0200
 U 1 1 52DEA2A1
 P 6850 3850
-F 0 "#PWR0191" H 6850 3940 20  0001 C CNN
+F 0 "#PWR0200" H 6850 3940 20  0001 C CNN
 F 1 "+5V" H 6850 3940 30  0000 C CNN
 F 2 "" H 6850 3850 60  0000 C CNN
@@
 $EndComp
 $Comp
-L +3.3V #PWR0192
+L +3.3V-RESCUE-ciaa-pic #PWR0201
 U 1 1 52DEA2B0
 P 8300 3850
-F 0 "#PWR0192" H 8300 3810 30  0001 C CNN
+F 0 "#PWR0201" H 8300 3810 30  0001 C CNN
 F 1 "+3.3V" H 8300 3960 30  0000 C CNN
 F 2 "" H 8300 3850 60  0000 C CNN
@@
 $EndComp
 $Comp
-L +3.3VADC #PWR0193
+L +3.3VADC #PWR0202
 U 1 1 52DEA2BF
 P 9500 3850
-F 0 "#PWR0193" H 9500 3970 20  0001 C CNN
+F 0 "#PWR0202" H 9500 3970 20  0001 C CNN
 F 1 "+3.3VADC" H 9500 3940 30  0000 C CNN
 F 2 "" H 9500 3850 60  0000 C CNN
@@
 $EndComp
 $Comp
-L GND #PWR0194
+L GND-RESCUE-ciaa-pic #PWR0203
 U 1 1 52DEAAB6
 P 8650 4900
-F 0 "#PWR0194" H 8650 4900 30  0001 C CNN
+F 0 "#PWR0203" H 8650 4900 30  0001 C CNN
 F 1 "GND" H 8650 4830 30  0001 C CNN
 F 2 "" H 8650 4900 60  0000 C CNN
@@
 	8650 4750 8700 4750
 $Comp
-L GNDA #PWR0195
+L GNDA-RESCUE-ciaa-pic #PWR0204
 U 1 1 52DEAAE6
 P 9500 4900
-F 0 "#PWR0195" H 9500 4900 40  0001 C CNN
+F 0 "#PWR0204" H 9500 4900 40  0001 C CNN
 F 1 "GNDA" H 9500 4830 40  0000 C CNN
 F 2 "" H 9500 4900 60  0000 C CNN
@@
 	9500 4750 9400 4750
 $Comp
-L PWR_FLAG #FLG0196
+L PWR_FLAG #FLG0205
 U 1 1 52DFF728
 P 7000 3850
-F 0 "#FLG0196" H 7000 3945 30  0001 C CNN
+F 0 "#FLG0205" H 7000 3945 30  0001 C CNN
 F 1 "PWR_FLAG" H 7000 4030 30  0000 C CNN
 F 2 "" H 7000 3850 60  0000 C CNN
@@
 Connection ~ 6850 3900
 $Comp
-L PWR_FLAG #FLG0197
+L PWR_FLAG #FLG0206
 U 1 1 52DFF757
 P 9750 3850
-F 0 "#FLG0197" H 9750 3945 30  0001 C CNN
+F 0 "#FLG0206" H 9750 3945 30  0001 C CNN
 F 1 "PWR_FLAG" H 9750 4030 30  0000 C CNN
 F 2 "" H 9750 3850 60  0000 C CNN
@@
 Connection ~ 9500 3900
 $Comp
-L PWR_FLAG #FLG0198
+L PWR_FLAG #FLG0207
 U 1 1 52DFF7BB
 P 9500 4700
-F 0 "#FLG0198" H 9500 4795 30  0001 C CNN
+F 0 "#FLG0207" H 9500 4795 30  0001 C CNN
 F 1 "PWR_FLAG" H 9500 4880 30  0000 C CNN
 F 2 "" H 9500 4700 60  0000 C CNN
@@
 	8650 4750 8650 4900
 $Comp
-L PWR_FLAG #FLG0199
+L PWR_FLAG #FLG0208
 U 1 1 52E04B0F
 P 2950 3600
-F 0 "#FLG0199" H 2950 3695 30  0001 C CNN
+F 0 "#FLG0208" H 2950 3695 30  0001 C CNN
 F 1 "PWR_FLAG" H 2950 3780 30  0000 C CNN
 F 2 "" H 2950 3600 60  0000 C CNN
@@
 	2900 4050 2900 4300
 $Comp
-L PWR_FLAG #FLG0200
+L PWR_FLAG #FLG0209
 U 1 1 52E04BC7
 P 2750 4300
-F 0 "#FLG0200" H 2750 4395 30  0001 C CNN
+F 0 "#FLG0209" H 2750 4395 30  0001 C CNN
 F 1 "PWR_FLAG" H 2750 4480 30  0000 C CNN
 F 2 "" H 2750 4300 60  0000 C CNN
@@
 Connection ~ 2750 4050
 $Comp
-L PWR_FLAG #FLG0201
+L PWR_FLAG #FLG0210
 U 1 1 52E0BE77
 P 5950 3250
-F 0 "#FLG0201" H 5950 3345 30  0001 C CNN
+F 0 "#FLG0210" H 5950 3345 30  0001 C CNN
 F 1 "PWR_FLAG" H 5950 3430 30  0000 C CNN
 F 2 "" H 5950 3250 60  0000 C CNN
@@
 	6400 2500 6550 2500
 $Comp
-L PWR_FLAG #FLG0202
+L PWR_FLAG #FLG0211
 U 1 1 52EACD34
 P 5950 2450
-F 0 "#FLG0202" H 5950 2545 30  0001 C CNN
+F 0 "#FLG0211" H 5950 2545 30  0001 C CNN
 F 1 "PWR_FLAG" H 5950 2630 30  0000 C CNN
 F 2 "" H 5950 2450 60  0000 C CNN
@@
 $EndComp
 $Comp
-L LED D25
+L LED-RESCUE-ciaa-pic D25
 U 1 1 551A51A4
 P 8150 5000
@@
 $EndComp
 $Comp
-L R R110
+L R-RESCUE-ciaa-pic R110
 U 1 1 551A51AA
 P 8150 4500
@@
 $EndComp
 $Comp
-L GND #PWR0203
+L GND-RESCUE-ciaa-pic #PWR0212
 U 1 1 551A51B0
 P 8150 5350
-F 0 "#PWR0203" H 8150 5350 30  0001 C CNN
+F 0 "#PWR0212" H 8150 5350 30  0001 C CNN
 F 1 "GND" H 8150 5280 30  0001 C CNN
 F 2 "" H 8150 5350 60  0000 C CNN

Commit message: elimino conector salida reles
Parts:
- C16, C17, C18, D1, D2, D25, D3, D4, D5, FB20, FB6, J18, L2, TH1, U3, U4, ZA1, ZA14: footprint ~ -> (none)
- R110, R22: footprint ~ -> Resistors_SMD:R_0603

Commit message: rev02 aignacion footprint
Parts:
- D25: footprint (none) -> LEDs:LED_0603
- J18: footprint (none) -> footprints:bornier2
Changed lines of the file:
@@
 F 0 "J18" H 2150 4200 60  0000 C CNN
 F 1 "TB_1X2" H 2250 3700 60  0000 C CNN
-F 2 "" H 2150 4000 60  0001 C CNN
+F 2 "footprints:bornier2" H 2150 4000 60  0001 C CNN
 F 3 "~" H 2150 4000 60  0000 C CNN
 	1    2200 3950
@@
 F 0 "D25" H 8150 5100 50  0000 C CNN
 F 1 "LED green" H 8150 4900 50  0000 C CNN
-F 2 "" H 8150 5000 60  0001 C CNN
+F 2 "LEDs:LED_0603" H 8150 5000 60  0001 C CNN
 F 3 "~" H 8150 5000 60  0000 C CNN
 	1    8150 5000

Commit message: rev02 se completa campo num. de frabicante(#manf) CIAA-PIC
Parts:
- C16: footprint (none) -> footprints:c_elec_13.7x13x13.5; #manf (none) -> UCL1V471MNL1GS
- C17: footprint (none) -> footprints:c_elec_6.3x7.7; #manf (none) -> UCW1C331MNL1GS
- C18: footprint (none) -> footprints:c_1206_tantalio; #manf (none) -> T491A106K006AT
- D1, D5: footprint (none) -> footprints:SOD323; #manf (none) -> PMEG3020EH,115
- D2: footprint (none) -> Diodes_SMD:DO-214AB; #manf (none) -> MURS360T3G
- D25: #manf (none) -> LTST-C191KGKT
- D3: footprint (none) -> footprints:DO-214AB(SMC); #manf (none) -> B540C-13-F
- D4: footprint (none) -> footprints:LED-0603; #manf (none) -> QTLP600C7TR
- FB20, FB6: footprint (none) -> footprints:SM0603_Resistor; #manf (none) -> MMZ1608B601CTAH0
- J18: #manf (none) -> OSTTC022162
- L2: footprint (none) -> footprints:Inductor_10x9.8mm; #manf (none) -> SRN1060-470M
- R110, R22: #manf (none) -> RC0603JR-071KL
- TH1: footprint (none) -> footprints:2-SMD-MF-SM030; #manf (none) -> MF-SM300-2
- U3: footprint (none) -> footprints:TO263-6--D2PACK5-LM2596; #manf (none) -> LM2596SX-5.0/NOPB
- U4: footprint (none) -> footprints:SOT223; #manf (none) -> NCP1117ST33T3G
- ZA1: footprint (none) -> footprints:DO214AA-1-2; #manf (none) -> P6SMB33CA-E3/52
- ZA14: footprint (none) -> footprints:SOD123F; #manf (none) -> MMSZ5V6T1G

Commit message: rev02 se completa campo num. de frabicante(manf#) CIAA-PIC
Parts:
- C16: #manf UCL1V471MNL1GS -> (none); manf# (none) -> UCL1V471MNL1GS
- C17: #manf UCW1C331MNL1GS -> (none); manf# (none) -> UCW1C331MNL1GS
- C18: #manf T491A106K006AT -> (none); manf# (none) -> T491A106K006AT
- D1, D5: #manf PMEG3020EH,115 -> (none); manf# (none) -> PMEG3020EH,115
- D2: #manf MURS360T3G -> (none); manf# (none) -> MURS360T3G
- D25: #manf LTST-C191KGKT -> (none); manf# (none) -> LTST-C191KGKT
- D3: #manf B540C-13-F -> (none); manf# (none) -> B540C-13-F
- D4: #manf QTLP600C7TR -> (none); manf# (none) -> QTLP600C7TR
- FB20, FB6: #manf MMZ1608B601CTAH0 -> (none); manf# (none) -> MMZ1608B601CTAH0
- J18: #manf OSTTC022162 -> (none); manf# (none) -> OSTTC022162
- L2: #manf SRN1060-470M -> (none); manf# (none) -> SRN1060-470M
- R110, R22: #manf RC0603JR-071KL -> (none); manf# (none) -> RC0603JR-071KL
- TH1: #manf MF-SM300-2 -> (none); manf# (none) -> MF-SM300-2
- U3: #manf LM2596SX-5.0/NOPB -> (none); manf# (none) -> LM2596SX-5.0/NOPB
- U4: #manf NCP1117ST33T3G -> (none); manf# (none) -> NCP1117ST33T3G
- ZA1: #manf P6SMB33CA-E3/52 -> (none); manf# (none) -> P6SMB33CA-E3/52
- ZA14: #manf MMSZ5V6T1G -> (none); manf# (none) -> MMSZ5V6T1G
Changed lines of the file:
@@
 F 2 "footprints:SOT223" H 7700 4300 60  0001 C CNN
 F 3 "~" H 7700 4300 60  0000 C CNN
-F 4 "NCP1117ST33T3G" H 7700 4300 60  0001 C CNN "#manf"
+F 4 "NCP1117ST33T3G" H 7700 4300 60  0001 C CNN "manf#"
 	1    7700 4300
 	1    0    0    -1
@@
 F 2 "footprints:TO263-6--D2PACK5-LM2596" H 5200 4050 60  0001 C CNN
 F 3 "~" H 5200 4050 60  0000 C CNN
-F 4 "LM2596SX-5.0/NOPB" H 5200 4050 60  0001 C CNN "#manf"
+F 4 "LM2596SX-5.0/NOPB" H 5200 4050 60  0001 C CNN "manf#"
 	1    5200 4050
 	1    0    0    -1
@@
 F 2 "footprints:c_elec_13.7x13x13.5" H 3850 3900 30  0001 C CNN
 F 3 "~" H 3750 4050 300 0000 C CNN
-F 4 "UCL1V471MNL1GS" H 3750 4050 60  0001 C CNN "#manf"
+F 4 "UCL1V471MNL1GS" H 3750 4050 60  0001 C CNN "manf#"
 	1    3750 4050
 	1    0    0    -1
@@
 F 2 "footprints:Inductor_10x9.8mm" H 6250 4250 60  0001 C CNN
 F 3 "~" H 6250 4250 60  0000 C CNN
-F 4 "SRN1060-470M " V 6250 4250 60  0001 C CNN "#manf"
+F 4 "SRN1060-470M " V 6250 4250 60  0001 C CNN "manf#"
 	1    6250 4250
 	0    -1   -1   0
@@
 F 2 "Diodes_SMD:DO-214AB" H 2900 3850 60  0001 C CNN
 F 3 "~" H 2900 3850 60  0000 C CNN
-F 4 " MURS360T3G " H 2900 3850 60  0001 C CNN "#manf"
+F 4 " MURS360T3G " H 2900 3850 60  0001 C CNN "manf#"
 	1    2900 3850
 	1    0    0    -1
@@
 F 2 "footprints:DO-214AB(SMC)" H 5850 4450 60  0001 C CNN
 F 3 "~" H 5850 4450 60  0000 C CNN
-F 4 "B540C-13-F " H 5850 4450 60  0001 C CNN "#manf"
+F 4 "B540C-13-F " H 5850 4450 60  0001 C CNN "manf#"
 	1    5850 4450
 	0    -1   -1   0
@@
 F 2 "footprints:c_elec_6.3x7.7" H 6950 4300 30  0001 C CNN
 F 3 "~" H 6850 4450 300 0000 C CNN
-F 4 "UCW1C331MNL1GS " H 6850 4450 60  0001 C CNN "#manf"
+F 4 "UCW1C331MNL1GS " H 6850 4450 60  0001 C CNN "manf#"
 	1    6850 4450
 	1    0    0    -1
@@
 F 2 "footprints:c_1206_tantalio" H 8500 4300 30  0001 C CNN
 F 3 "~" H 8400 4450 300 0000 C CNN
-F 4 "T491A106K006AT" H 8400 4450 60  0001 C CNN "#manf"
+F 4 "T491A106K006AT" H 8400 4450 60  0001 C CNN "manf#"
 	1    8400 4450
 	1    0    0    -1
@@
 F 2 "footprints:SOD323" H 6200 3300 60  0001 C CNN
 F 3 "~" H 6200 3300 60  0000 C CNN
-F 4 "PMEG3020EH,115 " H 6200 3300 60  0001 C CNN "#manf"
+F 4 "PMEG3020EH,115 " H 6200 3300 60  0001 C CNN "manf#"
 	1    6200 3300
 	1    0    0    -1
@@
 F 2 "footprints:2-SMD-MF-SM030" H 3450 3850 60  0001 C CNN
 F 3 "~" H 3450 3850 60  0000 C CNN
-F 4 "MF-SM300-2" V 3450 3850 60  0001 C CNN "#manf"
+F 4 "MF-SM300-2" V 3450 3850 60  0001 C CNN "manf#"
 	1    3450 3850
 	0    -1   -1   0
@@
 F 2 "footprints:DO214AA-1-2" H 4300 4100 60  0001 C CNN
 F 3 "~" H 4300 4100 60  0000 C CNN
-F 4 "P6SMB33CA-E3/52" H 4300 4100 60  0001 C CNN "#manf"
+F 4 "P6SMB33CA-E3/52" H 4300 4100 60  0001 C CNN "manf#"
 	1    4300 4100
 	0    1    1    0
@@
 F 2 "footprints:LED-0603" H 7150 5050 60  0001 C CNN
 F 3 "~" H 7150 5050 60  0000 C CNN
-F 4 "QTLP600C7TR" H 7150 5050 60  0001 C CNN "#manf"
+F 4 "QTLP600C7TR" H 7150 5050 60  0001 C CNN "manf#"
 	1    7150 5050
 	0    1    1    0
@@
 F 2 "Resistors_SMD:R_0603" V 7080 4550 30  0001 C CNN
 F 3 "~" H 7150 4550 30  0000 C CNN
-F 4 "RC0603JR-071KL" V 7150 4550 60  0001 C CNN "#manf"
+F 4 "RC0603JR-071KL" V 7150 4550 60  0001 C CNN "manf#"
 	1    7150 4550
 	1    0    0    -1
@@
 F 2 "footprints:SOD123F" H 6550 4550 60  0001 C CNN
 F 3 "~" H 6550 4550 60  0000 C CNN
-F 4 "MMSZ5V6T1G " H 6550 4550 60  0001 C CNN "#manf"
+F 4 "MMSZ5V6T1G " H 6550 4550 60  0001 C CNN "manf#"
 	1    6550 4550
 	0    1    1    0
@@
 F 2 "footprints:SM0603_Resistor" H 9050 4250 60  0001 C CNN
 F 3 "~" H 9050 4250 60  0000 C CNN
-F 4 "MMZ1608B601CTAH0" H 9050 4250 60  0001 C CNN "#manf"
+F 4 "MMZ1608B601CTAH0" H 9050 4250 60  0001 C CNN "manf#"
 	1    9050 4250
 	1    0    0    -1
@@
 F 2 "footprints:SM0603_Resistor" H 9050 4750 60  0001 C CNN
 F 3 "~" H 9050 4750 60  0000 C CNN
-F 4 "MMZ1608B601CTAH0" H 9050 4750 60  0001 C CNN "#manf"
+F 4 "MMZ1608B601CTAH0" H 9050 4750 60  0001 C CNN "manf#"
 	1    9050 4750
 	1    0    0    -1
@@
 F 2 "footprints:SOD323" H 6200 2500 60  0001 C CNN
 F 3 "~" H 6200 2500 60  0000 C CNN
-F 4 "PMEG3020EH,115 " H 6200 2500 60  0001 C CNN "#manf"
+F 4 "PMEG3020EH,115 " H 6200 2500 60  0001 C CNN "manf#"
 	1    6200 2500
 	1    0    0    -1
@@
 F 2 "footprints:bornier2" H 2150 4000 60  0001 C CNN
 F 3 "~" H 2150 4000 60  0000 C CNN
-F 4 "OSTTC022162" H 2200 3950 60  0001 C CNN "#manf"
+F 4 "OSTTC022162" H 2200 3950 60  0001 C CNN "manf#"
 	1    2200 3950
 	1    0    0    -1
@@
 F 2 "LEDs:LED_0603" H 8150 5000 60  0001 C CNN
 F 3 "~" H 8150 5000 60  0000 C CNN
-F 4 "LTST-C191KGKT" H 8150 5000 60  0001 C CNN "#manf"
+F 4 "LTST-C191KGKT" H 8150 5000 60  0001 C CNN "manf#"
 	1    8150 5000
 	0    1    1    0
@@
 F 2 "Resistors_SMD:R_0603" V 8080 4500 30  0001 C CNN
 F 3 "~" H 8150 4500 30  0000 C CNN
-F 4 "RC0603JR-071KL" V 8150 4500 60  0001 C CNN "#manf"
+F 4 "RC0603JR-071KL" V 8150 4500 60  0001 C CNN "manf#"
 	1    8150 4500
 	1    0    0    -1
