File: PCB/PIC/analog_out.sch (KiCad schematic (older format))
At the start: 27 parts, among them J19 TB_1X2, Q1 PBSS5240XF, Q14 BC817-40, U18 LM358, U21 MCP6022

Commit message: CIAA PIC footprints done
Connections:
- net at C95.2, R149.1: now also U21.3 (+)
- net at C84.1, R150.2, U21.1: now also U21.2 (-)
Changed lines of the file:
@@
 LIBS:lan_8740
 LIBS:Pic32MZ
+LIBS:mcp1416
+LIBS:fqt13n06l
 LIBS:ciaa-pic-cache
 EELAYER 27 0
@@
 Sheet 8 12
 Title "CIAA - Salida Analógica"
-Date "29 dec 2014"
+Date "7 sep 2015"
 Rev "1.0"
 Comp ""
@@
 $EndDescr
 $Comp
-L +24V #PWR146
+L +24V #PWR0148
 U 1 1 532CCE3B
 P 3600 4450
-F 0 "#PWR146" H 3600 4400 20  0001 C CNN
+F 0 "#PWR0148" H 3600 4400 20  0001 C CNN
 F 1 "+24V" H 3600 4550 30  0000 C CNN
 F 2 "" H 3600 4450 60  0000 C CNN
@@
 $EndComp
 $Comp
-L GNDA #PWR148
+L GNDA #PWR0149
 U 1 1 532CFB46
 P 4700 5600
-F 0 "#PWR148" H 4700 5600 40  0001 C CNN
+F 0 "#PWR0149" H 4700 5600 40  0001 C CNN
 F 1 "GNDA" H 4700 5530 40  0000 C CNN
 F 2 "" H 4700 5600 60  0000 C CNN
@@
 $EndComp
 $Comp
-L GNDA #PWR149
+L GNDA #PWR0150
 U 1 1 532CFB6F
 P 5250 4500
-F 0 "#PWR149" H 5250 4500 40  0001 C CNN
+F 0 "#PWR0150" H 5250 4500 40  0001 C CNN
 F 1 "GNDA" H 5250 4430 40  0000 C CNN
 F 2 "" H 5250 4500 60  0000 C CNN
@@
 $EndComp
 $Comp
-L GNDA #PWR147
+L GNDA #PWR0151
 U 1 1 532D06E5
 P 4000 6550
-F 0 "#PWR147" H 4000 6550 40  0001 C CNN
+F 0 "#PWR0151" H 4000 6550 40  0001 C CNN
 F 1 "GNDA" H 4000 6480 40  0000 C CNN
 F 2 "" H 4000 6550 60  0000 C CNN
@@
 $EndComp
 $Comp
-L GNDA #PWR158
+L GNDA #PWR0152
 U 1 1 532A8008
 P 8600 5800
-F 0 "#PWR158" H 8600 5800 40  0001 C CNN
+F 0 "#PWR0152" H 8600 5800 40  0001 C CNN
 F 1 "GNDA" H 8600 5730 40  0000 C CNN
 F 2 "" H 8600 5800 60  0000 C CNN
@@
 $EndComp
 $Comp
-L PWR_FLAG #FLG1
+L PWR_FLAG #FLG0153
 U 1 1 532B208A
 P 4700 4000
-F 0 "#FLG1" H 4700 4095 30  0001 C CNN
+F 0 "#FLG0153" H 4700 4095 30  0001 C CNN
 F 1 "PWR_FLAG" H 4700 4180 30  0000 C CNN
 F 2 "" H 4700 4000 60  0000 C CNN
@@
 $EndComp
 $Comp
-L GNDA #PWR157
+L GNDA #PWR0154
 U 1 1 532CECA5
 P 7800 4650
-F 0 "#PWR157" H 7800 4650 40  0001 C CNN
+F 0 "#PWR0154" H 7800 4650 40  0001 C CNN
 F 1 "GNDA" H 7800 4580 40  0000 C CNN
 F 2 "" H 7800 4650 60  0000 C CNN
@@
 $EndComp
 $Comp
-L GNDA #PWR156
+L GNDA #PWR0155
 U 1 1 532CF8E2
 P 7700 5700
-F 0 "#PWR156" H 7700 5700 40  0001 C CNN
+F 0 "#PWR0155" H 7700 5700 40  0001 C CNN
 F 1 "GNDA" H 7700 5630 40  0000 C CNN
 F 2 "" H 7700 5700 60  0000 C CNN
@@
 $EndComp
 $Comp
-L GNDA #PWR154
+L GNDA #PWR0156
 U 1 1 532CF93A
 P 6900 5700
-F 0 "#PWR154" H 6900 5700 40  0001 C CNN
+F 0 "#PWR0156" H 6900 5700 40  0001 C CNN
 F 1 "GNDA" H 6900 5630 40  0000 C CNN
 F 2 "" H 6900 5700 60  0000 C CNN
@@
 $EndComp
 $Comp
-L GNDA #PWR145
+L GNDA #PWR0157
 U 1 1 53BAF7F5
 P 2800 1650
-F 0 "#PWR145" H 2800 1650 40  0001 C CNN
+F 0 "#PWR0157" H 2800 1650 40  0001 C CNN
 F 1 "GNDA" H 2800 1580 40  0000 C CNN
 F 2 "" H 2800 1650 60  0000 C CNN
@@
 Ver AN538, AN655 Microchip\nMPLAB Started Kit for dsPIC (Fig A-6) \n
 $Comp
-L GNDA #PWR153
+L GNDA #PWR0158
 U 1 1 53BB004F
 P 6350 5550
-F 0 "#PWR153" H 6350 5550 40  0001 C CNN
+F 0 "#PWR0158" H 6350 5550 40  0001 C CNN
 F 1 "GNDA" H 6350 5480 40  0000 C CNN
 F 2 "" H 6350 5550 60  0000 C CNN
@@
 $EndComp
 $Comp
-L GNDA #PWR150
+L GNDA #PWR0159
 U 1 1 543D3CD6
 P 5300 2650
-F 0 "#PWR150" H 5300 2650 40  0001 C CNN
+F 0 "#PWR0159" H 5300 2650 40  0001 C CNN
 F 1 "GNDA" H 5300 2580 40  0000 C CNN
 F 2 "" H 5300 2650 60  0000 C CNN
@@
 $EndComp
 $Comp
-L GNDA #PWR155
+L GNDA #PWR0160
 U 1 1 543D3EA5
 P 7400 1500
-F 0 "#PWR155" H 7400 1500 40  0001 C CNN
+F 0 "#PWR0160" H 7400 1500 40  0001 C CNN
 F 1 "GNDA" H 7400 1430 40  0000 C CNN
 F 2 "" H 7400 1500 60  0000 C CNN
@@
 OUT
 $Comp
-L +3,3V #PWR151
+L +3,3V #PWR0161
 U 1 1 543D7CD7
 P 5900 1150
-F 0 "#PWR151" H 5900 1110 30  0001 C CNN
+F 0 "#PWR0161" H 5900 1110 30  0001 C CNN
 F 1 "+3,3V" H 5900 1260 30  0000 C CNN
 F 2 "" H 5900 1150 60  0000 C CNN
@@
 $EndComp
 $Comp
-L +3,3V #PWR144
+L +3,3V #PWR0162
 U 1 1 543D7CE4
 P 2800 1000
-F 0 "#PWR144" H 2800 960 30  0001 C CNN
+F 0 "#PWR0162" H 2800 960 30  0001 C CNN
 F 1 "+3,3V" H 2800 1110 30  0000 C CNN
 F 2 "" H 2800 1000 60  0000 C CNN
@@
 $EndComp
 $Comp
-L GNDA #PWR152
+L GNDA #PWR0163
 U 1 1 543D7CEA
 P 5900 2650
-F 0 "#PWR152" H 5900 2650 40  0001 C CNN
+F 0 "#PWR0163" H 5900 2650 40  0001 C CNN
 F 1 "GNDA" H 5900 2580 40  0000 C CNN
 F 2 "" H 5900 2650 60  0000 C CNN
@@
 	4450 1850 4700 1850
 Wire Wire Line
-	5200 1850 5450 1850
-Wire Wire Line
 	4600 1850 4600 1500
 Wire Wire Line
@@
 Connection ~ 4600 1850
 Wire Wire Line
-	6500 2450 5450 2450
-Wire Wire Line
-	5450 2450 5450 2050
+	6500 2450 5400 2450
 Connection ~ 6500 1950
 Wire Wire Line
@@
 Connection ~ 6900 1500
 Connection ~ 6500 1500
-Connection ~ 5450 1850
-Connection ~ 5450 2050
+Connection ~ 5400 1850
+Connection ~ 5400 2050
 Connection ~ 4700 1850
 Connection ~ 5050 1500
@@
 Wire Wire Line
 	5900 1550 5900 1150
+Wire Wire Line
+	5400 2450 5400 2050
+Wire Wire Line
+	5200 1850 5400 1850
+Connection ~ 5200 1850
+Connection ~ 5300 2150
+Connection ~ 5300 2550
+Connection ~ 5900 2350
+Connection ~ 6400 1950
 $EndSCHEMATC

Commit message: Correcciones al esquematico segun rev01
Parts:
- added D?: BAV199, symbol BAV199
- added TH?: MF-USMF005-2, symbol THERMISTOR
- C46, C66, C84, C88, C95, C96, C97: symbol C -> C-RESCUE-ciaa-pic
- J19: footprint ~ -> footprints:bornier2
- R105, R107, R109, R141, R148, R149, R150, R80, R82, R83: symbol R -> R-RESCUE-ciaa-pic
- U18: symbol LM358 -> LM358-RESCUE-ciaa-pic
Connections:
- net 24V_A: now also D?.1 (K)
- net GNDA: now also D?.3 (A)
- new net: D?.2 (KA), TH?.1
Other:
- note added: "24V_A Podría ser un símbolo de alimentación."
- note added: "D48. Línea de conexión cruza símbolo.\nDesprolijo."
- note added: "OUT podría conectarse.\nQue es cada bloque marcado?"
- moved on the sheet: C46, C66, C84, C88, C96, C97, D46, D48, FB21, J19, JP16, Q1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
