File: PCB/PIC/ciaa-pic.kicad_pcb (KiCad board)
At the start: 4 copper layers, 138.8 x 86.3 mm, 436 parts, among them IC1 PS2805-4, IC2 PS2805-4, J1 TB_1X3, J10 TB_1X3, J11 TB_1X2, J12 TB_1X3, J13 TB_1X3, J14 TB_1X2, J15 TB_1X3, J16 TB_1X3, J17 TB_1X2, J18 TB_1X2, J19 TB_1X2, J2 TB_1X3, J3 DB9, J4 TB_1X3, J5 RJ45-TRANSFO, J6 ZX62-AB-5PA, J7 ZX62-AB-5PA, J8 TB_1X3, J9 TB_1X3, K1 RELAY_TE_1461353-2, K2 RELAY_TE_1461353-2, K3 RELAY_TE_1461353-2, K4 RELAY_TE_1461353-2, P1 CONN_6X2, P14 SPI, P4 CONN_6, P6 CONN_4X2, Q1 PBSS5240XF, Q11 NDS7002A, Q12 NDS7002A, Q14 BC817-40, Q2 FQT13N06L, Q3 FQT13N06L, Q4 FQT13N06L, Q5 FQT13N06L, Q6 NDS7002A, Q7 NDS7002A, SW1 SW_PUSH_4, U1 LAN_8740, U10 MIC2025-2YM, U11 MCP6024, U12 24AA1025, U13 24AA025E48, U14 TXB0108, U16 PIC32MZ2048EC, U17 FT2232H, U18 LM358, U19 93C46, U2 SI502, U20 SST26VF064BA, U21 MCP6022, U22 ASDMB-24.000MHZ-LC-T, U23 MCP1416, U24 23A1024, U25 TC25L5I32K7680, U26 MCP9700, U27 MCP1416, U28 MCP1416, U29 MCP1416, U3 LM2596-5.0, U4 NCP1117ST33T3G, U5 MAX3072, U6 ST3232E, U7 VP231, U8 PESD1CAN, U9 PRTR5V0U2X, X1 FA-238V

Commit message: correcciones pcb
Parts:
- removed REF**: Measurement_Point_Round-SMD-Pad_Small, Measurement_Points:Measurement_Point_Round-SMD-Pad_Small
- D27: moved to B.Cu
- moved Q11 25.4 mm to (83.6, 74.1)
- moved R115 25.1 mm to (83.5, 77.0)
- moved D31 24.6 mm to (77.8, 69.7), turned to 180 degrees
- moved D30 24.0 mm to (87.5, 69.8)
- moved D27 22.8 mm to (66.8, 69.7), turned to 180 degrees
- moved Q12 22.1 mm to (72.9, 74.1)
- moved R116 21.9 mm to (72.8, 71.3)
- moved R111 21.1 mm to (62.4, 77.0), turned to 180 degrees
- moved Q6 21.1 mm to (62.3, 74.1)
- moved Q7 20.7 mm to (51.9, 74.1)
- moved R112 20.0 mm to (51.9, 71.3)
- moved D28 19.6 mm to (56.9, 69.7), turned to 180 degrees
- moved R113 4.96 mm to (54.7, 61.7), turned to 0 degrees
- moved R49 3.15 mm to (62.0, 55.4)
- moved ? 2.52 mm to (146.6, 29.4)
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Routing:
- net /USB OTG/USB0_PWR_FAULT: track 0.00 -> 116.6 mm, vias 0 -> 1
- net /CPU/CAN_TD: track 0.05 -> 87.5 mm, vias 0 -> 1
- net Net-(D30-Pad1): track 0.00 -> 62.0 mm, vias 0 -> 1
- net /CPU/DOUT7: track 3.91 -> 60.8 mm, vias 0 -> 1
- net Net-(C95-Pad2): track 0.39 -> 46.6 mm
- net /CPU/DOUT5: track 5.01 -> 49.4 mm, vias 0 -> 1
- net /CPU/GPIO3: track 0.00 -> 41.5 mm, vias 0 -> 2
- net /CPU/DOUT1: track 0.00 -> 35.8 mm, vias 0 -> 1
- net /GPIO/AN1: track 0.01 -> 33.2 mm, vias 0 -> 1
- net /GPIO/AN2: track 0.00 -> 32.5 mm, vias 0 -> 1
- net Net-(D23-Pad2): track 0.23 -> 31.2 mm, vias 0 -> 1
- net Net-(D31-Pad1): track 16.9 -> 46.7 mm
- net /JTAG/USB_JTAG_1.8V: track 33.1 -> 60.1 mm, vias 5 -> 6
- net /CPU/DOUT2: track 0.00 -> 26.1 mm, vias 0 -> 1
- net Net-(C84-Pad1): track 18.0 -> 42.7 mm
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- added copper zone on Inner2.Cu, net /JTAG/USB_JTAG_1.8V
- added copper zone on B.Cu, net Net-(C64-Pad1)
- added copper zone on F.Cu, net Net-(C64-Pad1)
- added copper zone on F.Cu, net Net-(FB7-Pad1)
- added copper zone on F.Cu, net Net-(Q2-Pad4)
- added copper zone on F.Cu, net Net-(Q3-Pad4)
- added copper zone on F.Cu, net Net-(Q4-Pad4)
- added copper zone on F.Cu, net Net-(Q5-Pad4)
- removed copper zone on Inner2.Cu, net /CPU/USB_JTAG_1.8V
- removed copper zone on F.Cu, net N-00000168
- removed copper zone on F.Cu, net N-00000377
- removed copper zone on F.Cu, net N-00000378
- removed copper zone on F.Cu, net N-00000379
- removed copper zone on F.Cu, net N-00000390

Commit message: correccion pcb
Parts:
- C9: moved to F.Cu
- moved C9 4.47 mm to (22.4, 79.5)
- moved D3 1.37 mm to (129.5, 78.2), turned to 180 degrees
- moved D2 0.12 mm to (128.2, 89.2), turned to 180 degrees
- turned C88 to 270 degrees
- renumbered F1 to ?, F2 to ?, F3 to ?, F4 to ?, F5 to ?, F6 to ?
Routing:
- net GND: track 485.9 -> 507.5 mm, vias 103 -> 106
- net /Salida Analógica/OUT: track 0.95 -> 18.7 mm, vias 0 -> 1
- net Net-(C95-Pad2): track 46.6 -> 63.8 mm
- net Net-(C97-Pad1): track 0.00 -> 11.6 mm
- net +3.3V: track 264.9 -> 275.1 mm, vias 61 -> 62
- net GNDA: track 124.6 -> 134.1 mm, vias 27 -> 30
- net Net-(D9-Pad2): track 4.28 -> 13.6 mm, vias 0 -> 2
- net Net-(C96-Pad2): track 7.29 -> 16.6 mm
- net Net-(D23-Pad2): track 31.2 -> 39.6 mm, vias 1 -> 2
- net Net-(D2-Pad1): track 0.49 -> 8.18 mm
- net Net-(C88-Pad2): track 0.51 -> 7.73 mm
- net (no net): track 6.49 -> 0.38 mm, vias 2 -> 0
- net +3.3VADC: track 46.8 -> 52.9 mm, vias 6 -> 7
- net +24V: track 15.4 -> 21.0 mm
- net Net-(D48-Pad2): track 6.99 -> 11.5 mm
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- added copper zone on B.Cu, net Net-(C16-Pad1)
- added copper zone on F.Cu, net Net-(C16-Pad1)
- added copper zone on B.Cu, net Net-(D2-Pad1)
- added copper zone on B.Cu, net Net-(D3-Pad2)
- added copper zone on F.Cu, net Net-(D3-Pad2)
- added copper zone on F.Cu, net Net-(FB1-Pad2)
- added copper zone on F.Cu, net Net-(J13-Pad1)
- added copper zone on F.Cu, net Net-(J13-Pad2)
- added copper zone on F.Cu, net Net-(J15-Pad2)
- added copper zone on F.Cu, net Net-(J15-Pad3)
- added copper zone on B.Cu, net Net-(J2-Pad1)
- added copper zone on B.Cu, net Net-(J2-Pad2)
- removed copper zone on F.Cu, net /USB OTG/GND_SH
- removed copper zone on B.Cu, net N-00000225
- removed copper zone on B.Cu, net N-00000226
- removed copper zone on B.Cu, net N-00000239
- removed copper zone on B.Cu, net N-00000240
- removed copper zone on F.Cu, net N-00000240
- removed copper zone on B.Cu, net N-00000241
- removed copper zone on F.Cu, net N-00000241
- removed copper zone on F.Cu, net N-00000373
- removed copper zone on F.Cu, net N-00000374
- removed copper zone on F.Cu, net N-00000375
- removed copper zone on F.Cu, net N-00000376

Commit message: correccion pcb
Parts:
- moved ? 90.1 mm to (77.6, 87.4), turned to 180 degrees
- moved ? 2.59 mm to (147.1, 26.9)
- moved R100 1.70 mm to (82.5, 53.1)
- moved C7 0.50 mm to (48.5, 62.6), turned to 180 degrees
- moved C8 0.35 mm to (50.7, 62.5)
- renumbered H4 to ?, H1 to ?, H2 to ?, H3 to ?
Routing:
- net Net-(D30-Pad1): track 62.0 -> 69.2 mm, vias 1 -> 2
- net Net-(D31-Pad1): track 46.7 -> 52.1 mm
- net Net-(D24-Pad2): track 20.6 -> 25.8 mm, vias 1 -> 2
- net /CPU/DOUT2: track 26.1 -> 31.1 mm
- net +5V: track 131.9 -> 136.0 mm, vias 15 -> 16
- net Net-(D6-Pad1): track 34.9 -> 38.3 mm
- net /USB OTG/USB0_PWR_FAULT: track 116.6 -> 119.5 mm
- net /CPU/ENET_TX_EN: track 50.8 -> 48.5 mm
- net Net-(D6-Pad2): track 48.6 -> 50.9 mm
- net Net-(J2-Pad2): track 3.75 -> 1.72 mm, vias 1 -> 0
- net Net-(J2-Pad1): track 3.96 -> 1.93 mm, vias 1 -> 0
- net /CPU/DOUT0: track 27.1 -> 29.1 mm
- net +3.3V: track 275.1 -> 276.9 mm
- net /CPU/DOUT1: track 35.8 -> 34.3 mm
- net Net-(C7-Pad1): track 5.54 -> 6.85 mm
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- added copper zone on B.Cu, net Net-(J15-Pad1)
- removed copper zone on B.Cu, net N-00000356
- removed copper zone on F.Cu, net Net-(D6-Pad1)
- removed copper zone on F.Cu, net Net-(D6-Pad2)
Other:
- board text added: "3.3v"
- board text added: "5v"
- board text added: "CIAA PIC v1.0 8/2/2016 www.proyecto-ciaa.com.ar"
- board text added: "JTAG-Debug"
- board text added: "OTG"
- board text added: "R.term RS485"
- board text added: "Rx"
- board text added: "Tx"
- board text removed: "CIAA Microchip PI32MZ v1.0 8/2/2016 www.proyecto-ciaa.com.ar"

Commit message: correccion pcb
Parts:
- C3: moved to B.Cu
- R3, R4, R5, R6: moved to F.Cu
- moved R5 20.5 mm to (42.8, 60.8), turned to 90 degrees
- moved R6 20.4 mm to (40.0, 60.1), turned to 90 degrees
- moved R3 18.8 mm to (38.4, 60.1), turned to 90 degrees
- moved R4 11.9 mm to (38.1, 55.2)
- moved ? 7.56 mm to (140.6, 36.6)
- moved ? 7.55 mm to (140.6, 36.6)
- moved ? 5.14 mm to (142.1, 28.2)
- moved L1 4.83 mm to (42.1, 63.3)
- moved C3 2.61 mm to (40.2, 61.7), turned to 90 degrees
- moved R19 2.22 mm to (42.8, 63.7)
- moved ? 0.95 mm to (28.3, 53.9)
- moved ? 0.93 mm to (28.3, 53.9)
- moved ? 0.65 mm to (77.8, 86.8)
Routing:
- net /Ethernet/+Filter: track 75.1 -> 61.0 mm, vias 4 -> 5
- net Net-(C12-Pad1): track 29.6 -> 27.1 mm
- net Net-(R19-Pad1): track 3.74 -> 5.63 mm
- net Net-(C14-Pad1): track 43.3 -> 44.9 mm
- net Net-(C11-Pad1): track 31.7 -> 30.2 mm
- net Net-(C13-Pad1): track 39.8 -> 41.1 mm
- net /Ethernet/LED_LINK: track 18.7 -> 19.9 mm
- net /Ethernet/LED_100M: track 16.1 -> 16.9 mm
- net GND: track 508.7 -> 508.0 mm
- net Net-(Q14-Pad3): track 15.8 -> 15.2 mm
- net +3.3V: track 276.9 -> 277.4 mm
- net (no net): track 0.32 -> 0.09 mm, vias 0 -> 1
