File: PCB/Safety/BUS_ISA.sch (KiCad schematic (older format))
At the start: 58 parts, among them P7 CONN_02X32

Commit message: Added Diego Fusari's last version. Changes in texts, title blocks and sheet names.
Parts:
- D10, D12, D13, D14, D15, D16, D17, D18, D19, D21, D22, D24, D25, D26, D29, D30, D31, D32, D33, D34, D35, D36, D37, D38, D40, D41, D42, D43, D45, D46, D47, D48, D49, D50, D51, D52, D53, D54, D55, D56, D57, D58, D60, D61: symbol BAV199 -> CIAA_Safety_VTI_1.0-rescue:BAV199
- P7: symbol CONN_02X32 -> CIAA_Safety_VTI_1.0-rescue:CONN_02X32
- R68, R69, R70, R71, R72, R73, R74, R75, R76, R77, R78, R79, R80: symbol R -> CIAA_Safety_VTI_1.0-rescue:R
