File: PCB/Safety/CAN.sch (KiCad schematic (older format))
At the start: 26 parts, among them U1 SN65HVD1040, U2 PESD1CAN, U3 SN65HVD1040, U4 PESD1CAN

Commit message: New version (-4) from Fusari,s Drive.
Parts:
- removed JP2, JP3, JP4, JP5: JUMPER, pin_array_x1:1X02, symbol JUMPER
- added P2: CAN 2, w_conn_mkds:mkds_1,5-3, symbol CONN_01X03
- added P3: CAN 1, w_conn_mkds:mkds_1,5-3, symbol CONN_01X03
- added P8: CAN2, w_pin_strip:pin_socket_2x2, symbol CONN_02X02
- added P9: CAN1, w_pin_strip:pin_socket_2x2, symbol CONN_02X02
- C1, C4: footprint w_smd_cap:c_tant_B -> w_smd_cap:c_tant_A; Digikey (none) -> 399-3685-1-ND
- C2, C3, C5, C6: Digikey (none) -> 478-5266-1-ND
- R1, R7: Digikey (none) -> P270AGCT-ND
- R10, R3, R4, R9: Digikey (none) -> 311-1.5KGRCT-ND
- R11, R12, R5, R6: Digikey (none) -> 311-60.4HRCT-ND
- R2, R8: Digikey (none) -> P4.70KABCT-ND
- U1, U3: Digikey (none) -> 296-21804-1-ND
- U2, U4: Digikey (none) -> 1727-3817-1-ND
Connections:
- wire segments 66 -> 92
Other:
- note added: "1%"
- note added: "Reemplazo\nAIMS42665TJAA1RG"

Commit message: Added Diego Fusari's last version. Changes in texts, title blocks and sheet names.
Parts:
- C1, C4: symbol CP1 -> CIAA_Safety_VTI_1.0-rescue:CP1
- C2, C3, C5, C6: symbol C -> CIAA_Safety_VTI_1.0-rescue:C
- P2, P3: symbol CONN_01X03 -> CIAA_Safety_VTI_1.0-rescue:CONN_01X03
- P8, P9: symbol CONN_02X02 -> CIAA_Safety_VTI_1.0-rescue:CONN_02X02
- R1, R10, R2, R3, R4, R7, R8, R9: symbol R -> CIAA_Safety_VTI_1.0-rescue:R
- R11, R12, R5, R6: value 60 -> 60-1%; symbol R -> CIAA_Safety_VTI_1.0-rescue:R
- U1, U3: symbol SN65HVD1040 -> CIAA_Safety_VTI_1.0-rescue:SN65HVD1040
- U2, U4: symbol PESD1CAN -> CIAA_Safety_VTI_1.0-rescue:PESD1CAN
Other:
- note removed: "1%"
