File: PCB/Safety/CIAA_Safety_VTI_1.0.sch (KiCad schematic (older format))
At the start: 6 parts, among them P1 JTAG

Commit message: New version (-4) from Fusari,s Drive.
Parts:
- removed PA1, PB1, PC1, PD1: CONN_01X30, w_pin_strip:pin_socket_2mm_30, symbol CONN_01X30
- JP1: footprint pin_array_x1:1X03 -> w_pin_strip:pin_strip_3; Digikey (none) -> 952-2263-ND
Connections:
- net labels added: INT_A, ISA_AD1IN[0], ISA_AD1IN[10], ISA_AD1IN[11], ISA_AD1IN[12], ISA_AD1IN[1], ISA_AD1IN[2], ISA_AD1IN[3], ISA_AD1IN[4], ISA_AD1IN[5], ISA_AD1IN[6], ISA_AD1IN[7], ISA_AD1IN[8], ISA_AD1IN[9], ISA_GPIO0, ISA_GPIO0/RESET_ETH, ISA_GPIO1, ISA_GPIO10, ISA_GPIO11, ISA_GPIO12, ISA_GPIO13, ISA_GPIO14, ISA_GPIO15, ISA_GPIO16, ISA_GPIO17, ISA_GPIO18, ISA_GPIO19, ISA_GPIO2, ISA_GPIO20, ISA_GPIO21, ISA_GPIO22, ISA_GPIO23, ISA_GPIO24, ISA_GPIO3, ISA_GPIO4, ISA_GPIO5, ISA_I2C_SCL, ISA_I2C_SDA, ISA_LINRX/GPIO35, ISA_LINTX/GPIO36, ISA_MIBSPI3CLK/GPIO32, ISA_MIBSPI3NCS[0]/GPIO34, ISA_MIBSPI3NCS[4]/GPIO27, ISA_MIBSPI3NCS[5]/GPIO33, ISA_MIBSPI3SIMO/GPIO31, ISA_MIBSPI3SOMI/GPIO30, ISA_MR, ISA_SCIRX/GPIO28, ISA_SCITX/GPIO29, ISA_nERROR, ISA_nRST, RSTI_A, V_MONITOR
- net labels removed: +12V, +5V, -12V, PCI_AD1IN[0], PCI_AD1IN[10], PCI_AD1IN[11], PCI_AD1IN[12], PCI_AD1IN[1], PCI_AD1IN[2], PCI_AD1IN[3], PCI_AD1IN[4], PCI_AD1IN[5], PCI_AD1IN[6], PCI_AD1IN[7], PCI_AD1IN[8], PCI_AD1IN[9], PCI_ADREFHI, PCI_ADREFLO, PCI_CAN1_H, PCI_CAN1_L, PCI_CAN2_H, PCI_CAN2_L, PCI_ETH_RXN, PCI_ETH_RXP, PCI_ETH_TXN, PCI_ETH_TXP, PCI_GPIO0, PCI_GPIO0/RESET_ETH, PCI_GPIO1, PCI_GPIO10, PCI_GPIO11, PCI_GPIO12, PCI_GPIO13, PCI_GPIO14, PCI_GPIO15, PCI_GPIO16, PCI_GPIO17, PCI_GPIO18, PCI_GPIO19, PCI_GPIO2, PCI_GPIO20, PCI_GPIO21, PCI_GPIO22, PCI_GPIO23, PCI_GPIO24, PCI_GPIO3, PCI_GPIO4, PCI_GPIO5, PCI_GPIO6, PCI_GPIO7, PCI_GPIO8, PCI_GPIO9, PCI_I2C_SCL/GPIO25, PCI_I2C_SDA/GPIO26, PCI_LED_ACT, PCI_LED_LINK, PCI_LINRX/GPIO35, PCI_LINTX/GPIO36, PCI_MIBSPI3CLK/GPIO32, PCI_MIBSPI3NCS[0]/GPIO34, PCI_MIBSPI3NCS[4]/GPIO27, PCI_MIBSPI3NCS[5]/GPIO33, PCI_MIBSPI3SIMO/GPIO31, PCI_MIBSPI3SOMI/GPIO30, PCI_MR, PCI_SCIRX/GPIO28, PCI_SCITX/GPIO29, PCI_VCCAD, PCI_nERROR, PCI_nRST, ground, pwr_+12, pwr_+3.3, pwr_+5, pwr_-12, pwr_vccad
- wire segments 222 -> 144
- no-connect marks 11 -> 3
Other:
- note added: "1. DIAGRAMA JERARQUICO"
- note added: "2. CAN 1/2"
- note added: "3. MEMORIA FLASH SPI"
- note added: "4. ETHERNET"
- note added: "5. CPU"
- note added: "6. USB OTG"
- note added: "7. USB HOST"
- note added: "8. BUS ISA"
- note added: "APLICACIONES AERONAUTICAS"
- note added: "Índice:"
- note removed: "BUS PCI-104"
- note removed: "VI/O"
- moved on the sheet: JP1, P1

Commit message: Added Diego Fusari's last version. Changes in texts, title blocks and sheet names.
Parts:
- JP1: symbol JUMPER3 -> CIAA_Safety_VTI_1.0-rescue:JUMPER3
- P1: symbol CONN_02X07 -> CIAA_Safety_VTI_1.0-rescue:CONN_02X07
Changed lines of the file:
@@
-EESchema Schematic File Version 2
-LIBS:74xgxx
-LIBS:74xx
-LIBS:ac-dc
-LIBS:actel
-LIBS:adc-dac
-LIBS:Altera
-LIBS:analog_devices
-LIBS:analog_switches
-LIBS:atmel
-LIBS:audio
-LIBS:brooktre
-LIBS:cmos_ieee
-LIBS:cmos4000
-LIBS:conn
-LIBS:contrib
-LIBS:cypress
-LIBS:dc-dc
-LIBS:device
-LIBS:digital-audio
-LIBS:diode
-LIBS:display
-LIBS:dsp
-LIBS:elec-unifil
-LIBS:ESD_Protection
-LIBS:ftdi
-LIBS:gennum
-LIBS:graphic
-LIBS:hc11
-LIBS:intel
-LIBS:interface
-LIBS:ir
-LIBS:Lattice
-LIBS:linear
-LIBS:logo
-LIBS:maxim
-LIBS:memory
-LIBS:microchip
-LIBS:microchip_dspic33dsc
-LIBS:microchip_pic10mcu
-LIBS:microchip_pic12mcu
-LIBS:microchip_pic16mcu
-LIBS:microchip_pic18mcu
-LIBS:microchip_pic32mcu
-LIBS:microcontrollers
-LIBS:motor_drivers
-LIBS:motorola
-LIBS:msp430
-LIBS:nordicsemi
-LIBS:nxp_armmcu
-LIBS:onsemi
-LIBS:opto
-LIBS:Oscillators
-LIBS:philips
-LIBS:power
-LIBS:Power_Management
-LIBS:powerint
-LIBS:pspice
-LIBS:references
-LIBS:regul
-LIBS:relays
-LIBS:rfcom
-LIBS:sensors
-LIBS:silabs
-LIBS:siliconi
-LIBS:stm8
-LIBS:stm32
-LIBS:supertex
-LIBS:switches
-LIBS:texas
-LIBS:transf
-LIBS:transistors
-LIBS:ttl_ieee
-LIBS:valves
-LIBS:video
-LIBS:Xicor
-LIBS:xilinx
-LIBS:Zilog
+EESchema Schematic File Version 4
 LIBS:CIAA_Safety_VTI_1.0-cache
-EELAYER 25 0
+EELAYER 30 0
 EELAYER END
 $Descr A4 11693 8268
 encoding utf-8
 Sheet 1 8
-Title "MODULO PROCESADOR SAFETY"
+Title "MÓDULO PROCESADOR SAFETY"
 Date "2015-12-15"
 Rev "1.0"
@@
 ISA_MR
 $Comp
-L JUMPER3 JP1
+L CIAA_Safety_VTI_1.0-rescue:JUMPER3 JP1
 U 1 1 56E6345D
 P 7010 1650
@@
 nTRST
 $Comp
-L +3.3V #PWR01
+L power:+3.3V #PWR01
 U 1 1 56F6A5B6
 P 1400 1520
@@
 $EndComp
 $Comp
-L CONN_02X07 P1
+L CIAA_Safety_VTI_1.0-rescue:CONN_02X07 P1
 U 1 1 56D0BED3
 P 1850 1620
@@
 NoConn ~ 2100 1520
 $Comp
-L GND #PWR02
+L power:GND #PWR02
 U 1 1 56D293A5
 P 2220 2080
@@
 	2100 1620 2220 1620
 Wire Wire Line
-	2220 1420 2220 2080
+	2220 1420 2220 1620
 Wire Wire Line
 	2220 1720 2100 1720
@@
 Text Notes 3200 1340 0    158  ~ 32
 APLICACIONES AERONAUTICAS
+Wire Wire Line
+	2220 1720 2220 1820
+Wire Wire Line
+	2220 1820 2220 2080
+Wire Wire Line
+	2220 1620 2220 1720
 $EndSCHEMATC
